File: PCB/ledmatrix.sch (KiCad schematic (older format))
At the start: 64 parts

Commit message: Add WIP yaemk 1.2 files
Parts:
- added D28, D33, D8: APA102-2020, prettylib:LED-APA102-2020, symbol LED:APA102-2020
- S10, S11, S12, S13, S14, S15, S16, S17, S18, S19, S2, S20, S21, S22, S24, S25, S26, S27, S28, S29, S3, S30, S31, S32, S33, S34, S35, S4, S9: footprint prettylib:MX_KAILH_SOCKET_WS2812_1U -> prettylib:MX_KAILH_SOCKET_SK9822_1U
Connections:
- wire segments 165 -> 175
Changed lines of the file:
@@
 F 0 "S28" V 3950 1550 50  0000 C CNN
 F 1 "SW" V 3950 1850 50  0000 C CNN
-F 2 "prettylib:MX_KAILH_SOCKET_WS2812_1U" H 4200 2150 60  0001 C CNN
+F 2 "prettylib:MX_KAILH_SOCKET_SK9822_1U" H 4200 2150 60  0001 C CNN
 F 3 "" H 4200 2150 60  0000 C CNN
 	2    4200 2150
@@
 F 0 "S21" V 6550 1550 50  0000 C CNN
 F 1 "SW" V 6550 1850 50  0000 C CNN
-F 2 "prettylib:MX_KAILH_SOCKET_WS2812_1U" H 6800 2150 60  0001 C CNN
+F 2 "prettylib:MX_KAILH_SOCKET_SK9822_1U" H 6800 2150 60  0001 C CNN
 F 3 "" H 6800 2150 60  0000 C CNN
 	2    6800 2150
@@
 F 0 "S14" V 7850 1550 50  0000 C CNN
 F 1 "SW" V 7850 1850 50  0000 C CNN
-F 2 "prettylib:MX_KAILH_SOCKET_WS2812_1U" H 8100 2150 60  0001 C CNN
+F 2 "prettylib:MX_KAILH_SOCKET_SK9822_1U" H 8100 2150 60  0001 C CNN
 F 3 "" H 8100 2150 60  0000 C CNN
 	2    8100 2150
@@
 F 0 "S3" V 9150 2300 50  0000 C CNN
 F 1 "SW" V 9150 2600 50  0000 C CNN
-F 2 "prettylib:MX_KAILH_SOCKET_WS2812_1U" H 9400 2900 60  0001 C CNN
+F 2 "prettylib:MX_KAILH_SOCKET_SK9822_1U" H 9400 2900 60  0001 C CNN
 F 3 "" H 9400 2900 60  0000 C CNN
 	2    9400 2900
@@
 F 0 "S12" V 7850 4700 50  0000 C CNN
 F 1 "SW" V 7850 5000 50  0000 C CNN
-F 2 "prettylib:MX_KAILH_SOCKET_WS2812_1U" H 8100 5300 60  0001 C CNN
+F 2 "prettylib:MX_KAILH_SOCKET_SK9822_1U" H 8100 5300 60  0001 C CNN
 F 3 "" H 8100 5300 60  0000 C CNN
 	2    8100 5300
@@
 F 0 "S15" V 6550 4700 50  0000 C CNN
 F 1 "SW" V 6550 5000 50  0000 C CNN
-F 2 "prettylib:MX_KAILH_SOCKET_WS2812_1U" H 6800 5300 60  0001 C CNN
+F 2 "prettylib:MX_KAILH_SOCKET_SK9822_1U" H 6800 5300 60  0001 C CNN
 F 3 "" H 6800 5300 60  0000 C CNN
 	2    6800 5300
@@
 F 0 "S20" V 5250 4700 50  0000 C CNN
 F 1 "SW" V 5250 5000 50  0000 C CNN
-F 2 "prettylib:MX_KAILH_SOCKET_WS2812_1U" H 5500 5300 60  0001 C CNN
+F 2 "prettylib:MX_KAILH_SOCKET_SK9822_1U" H 5500 5300 60  0001 C CNN
 F 3 "" H 5500 5300 60  0000 C CNN
 	2    5500 5300
@@
 F 0 "S27" V 3950 4700 50  0000 C CNN
 F 1 "SW" V 3950 5000 50  0000 C CNN
-F 2 "prettylib:MX_KAILH_SOCKET_WS2812_1U" H 4200 5300 60  0001 C CNN
+F 2 "prettylib:MX_KAILH_SOCKET_SK9822_1U" H 4200 5300 60  0001 C CNN
 F 3 "" H 4200 5300 60  0000 C CNN
 	2    4200 5300
@@
 F 0 "S11" V 7850 3850 50  0000 C CNN
 F 1 "SW" V 7850 4150 50  0000 C CNN
-F 2 "prettylib:MX_KAILH_SOCKET_WS2812_1U" H 8100 4450 60  0001 C CNN
+F 2 "prettylib:MX_KAILH_SOCKET_SK9822_1U" H 8100 4450 60  0001 C CNN
 F 3 "" H 8100 4450 60  0000 C CNN
 	2    8100 4450
@@
 F 0 "S16" V 6550 3850 50  0000 C CNN
 F 1 "SW" V 6550 4150 50  0000 C CNN
-F 2 "prettylib:MX_KAILH_SOCKET_WS2812_1U" H 6800 4450 60  0001 C CNN
+F 2 "prettylib:MX_KAILH_SOCKET_SK9822_1U" H 6800 4450 60  0001 C CNN
 F 3 "" H 6800 4450 60  0000 C CNN
 	2    6800 4450
@@
 F 0 "S19" V 5250 3850 50  0000 C CNN
 F 1 "SW" V 5250 4150 50  0000 C CNN
-F 2 "prettylib:MX_KAILH_SOCKET_WS2812_1U" H 5500 4450 60  0001 C CNN
+F 2 "prettylib:MX_KAILH_SOCKET_SK9822_1U" H 5500 4450 60  0001 C CNN
 F 3 "" H 5500 4450 60  0000 C CNN
 	2    5500 4450
@@
 F 0 "S31" V 3950 3850 50  0000 C CNN
 F 1 "SW" V 3950 4150 50  0000 C CNN
-F 2 "prettylib:MX_KAILH_SOCKET_WS2812_1U" H 4200 4450 60  0001 C CNN
+F 2 "prettylib:MX_KAILH_SOCKET_SK9822_1U" H 4200 4450 60  0001 C CNN
 F 3 "" H 4200 4450 60  0000 C CNN
 	2    4200 4450
@@
 F 0 "S10" V 7850 3050 50  0000 C CNN
 F 1 "SW" V 7850 3350 50  0000 C CNN
-F 2 "prettylib:MX_KAILH_SOCKET_WS2812_1U" H 8100 3650 60  0001 C CNN
+F 2 "prettylib:MX_KAILH_SOCKET_SK9822_1U" H 8100 3650 60  0001 C CNN
 F 3 "" H 8100 3650 60  0000 C CNN
 	2    8100 3650
@@
 F 0 "S17" V 6550 3050 50  0000 C CNN
 F 1 "SW" V 6550 3350 50  0000 C CNN
-F 2 "prettylib:MX_KAILH_SOCKET_WS2812_1U" H 6800 3650 60  0001 C CNN
+F 2 "prettylib:MX_KAILH_SOCKET_SK9822_1U" H 6800 3650 60  0001 C CNN
 F 3 "" H 6800 3650 60  0000 C CNN
 	2    6800 3650
@@
 F 0 "S24" V 5250 3050 50  0000 C CNN
 F 1 "SW" V 5250 3350 50  0000 C CNN
-F 2 "prettylib:MX_KAILH_SOCKET_WS2812_1U" H 5500 3650 60  0001 C CNN
+F 2 "prettylib:MX_KAILH_SOCKET_SK9822_1U" H 5500 3650 60  0001 C CNN
 F 3 "" H 5500 3650 60  0000 C CNN
 	2    5500 3650
@@
 F 0 "S30" V 3950 3050 50  0000 C CNN
 F 1 "SW" V 3950 3350 50  0000 C CNN
-F 2 "prettylib:MX_KAILH_SOCKET_WS2812_1U" H 4200 3650 60  0001 C CNN
+F 2 "prettylib:MX_KAILH_SOCKET_SK9822_1U" H 4200 3650 60  0001 C CNN
 F 3 "" H 4200 3650 60  0000 C CNN
 	2    4200 3650
@@
 F 0 "S9" V 7850 2300 50  0000 C CNN
 F 1 "SW" V 7850 2600 50  0000 C CNN
-F 2 "prettylib:MX_KAILH_SOCKET_WS2812_1U" H 8100 2900 60  0001 C CNN
+F 2 "prettylib:MX_KAILH_SOCKET_SK9822_1U" H 8100 2900 60  0001 C CNN
 F 3 "" H 8100 2900 60  0000 C CNN
 	2    8100 2900
@@
 F 0 "S22" V 6550 2300 50  0000 C CNN
 F 1 "SW" V 6550 2600 50  0000 C CNN
-F 2 "prettylib:MX_KAILH_SOCKET_WS2812_1U" H 6800 2900 60  0001 C CNN
+F 2 "prettylib:MX_KAILH_SOCKET_SK9822_1U" H 6800 2900 60  0001 C CNN
 F 3 "" H 6800 2900 60  0000 C CNN
 	2    6800 2900
@@
 F 0 "S25" V 5250 2300 50  0000 C CNN
 F 1 "SW" V 5250 2600 50  0000 C CNN
-F 2 "prettylib:MX_KAILH_SOCKET_WS2812_1U" H 5500 2900 60  0001 C CNN
+F 2 "prettylib:MX_KAILH_SOCKET_SK9822_1U" H 5500 2900 60  0001 C CNN
 F 3 "" H 5500 2900 60  0000 C CNN
 	2    5500 2900
@@
 F 0 "S29" V 3950 2300 50  0000 C CNN
 F 1 "SW" V 3950 2600 50  0000 C CNN
-F 2 "prettylib:MX_KAILH_SOCKET_WS2812_1U" H 4200 2900 60  0001 C CNN
+F 2 "prettylib:MX_KAILH_SOCKET_SK9822_1U" H 4200 2900 60  0001 C CNN
 F 3 "" H 4200 2900 60  0000 C CNN
 	2    4200 2900
@@
 F 0 "S35" V 2650 2300 50  0000 C CNN
 F 1 "SW" V 2650 2600 50  0000 C CNN
-F 2 "prettylib:MX_KAILH_SOCKET_WS2812_1U" H 2900 2900 60  0001 C CNN
+F 2 "prettylib:MX_KAILH_SOCKET_SK9822_1U" H 2900 2900 60  0001 C CNN
 F 3 "" H 2900 2900 60  0000 C CNN
 	2    2900 2900
@@
 F 0 "S34" V 2650 3050 50  0000 C CNN
 F 1 "SW" V 2650 3350 50  0000 C CNN
-F 2 "prettylib:MX_KAILH_SOCKET_WS2812_1U" H 2900 3650 60  0001 C CNN
+F 2 "prettylib:MX_KAILH_SOCKET_SK9822_1U" H 2900 3650 60  0001 C CNN
 F 3 "" H 2900 3650 60  0000 C CNN
 	2    2900 3650
@@
 F 0 "S33" V 2650 3850 50  0000 C CNN
 F 1 "SW" V 2650 4150 50  0000 C CNN
-F 2 "prettylib:MX_KAILH_SOCKET_WS2812_1U" H 2900 4450 60  0001 C CNN
+F 2 "prettylib:MX_KAILH_SOCKET_SK9822_1U" H 2900 4450 60  0001 C CNN
 F 3 "" H 2900 4450 60  0000 C CNN
 	2    2900 4450
@@
 F 0 "S32" V 2650 4700 50  0000 C CNN
 F 1 "SW" V 2650 5000 50  0000 C CNN
-F 2 "prettylib:MX_KAILH_SOCKET_WS2812_1U" H 2900 5300 60  0001 C CNN
+F 2 "prettylib:MX_KAILH_SOCKET_SK9822_1U" H 2900 5300 60  0001 C CNN
 F 3 "" H 2900 5300 60  0000 C CNN
 	2    2900 5300
@@
 F 0 "S18" V 2650 1550 50  0000 C CNN
 F 1 "SW" V 2650 1850 50  0000 C CNN
-F 2 "prettylib:MX_KAILH_SOCKET_WS2812_1U" H 2900 2150 60  0001 C CNN
+F 2 "prettylib:MX_KAILH_SOCKET_SK9822_1U" H 2900 2150 60  0001 C CNN
 F 3 "" H 2900 2150 60  0000 C CNN
 	2    2900 2150
@@
 F 0 "S13" V 1350 4750 50  0000 C CNN
 F 1 "SW" V 1350 5000 50  0000 C CNN
-F 2 "prettylib:MX_KAILH_SOCKET_WS2812_1U" H 1600 5300 60  0001 C CNN
+F 2 "prettylib:MX_KAILH_SOCKET_SK9822_1U" H 1600 5300 60  0001 C CNN
 F 3 "" H 1600 5300 60  0000 C CNN
 	2    1600 5300
@@
 F 0 "S26" V 5250 1550 50  0000 C CNN
 F 1 "SW" V 5250 1850 50  0000 C CNN
-F 2 "prettylib:MX_KAILH_SOCKET_WS2812_1U" H 5500 2150 60  0001 C CNN
+F 2 "prettylib:MX_KAILH_SOCKET_SK9822_1U" H 5500 2150 60  0001 C CNN
 F 3 "" H 5500 2150 60  0000 C CNN
 	2    5500 2150
@@
 F 0 "S4" V 9150 1550 50  0000 C CNN
 F 1 "SW" V 9150 1850 50  0000 C CNN
-F 2 "prettylib:MX_KAILH_SOCKET_WS2812_1U" H 9400 2150 60  0001 C CNN
+F 2 "prettylib:MX_KAILH_SOCKET_SK9822_1U" H 9400 2150 60  0001 C CNN
 F 3 "" H 9400 2150 60  0000 C CNN
 	2    9400 2150
@@
 F 0 "S2" V 9150 3050 50  0000 C CNN
 F 1 "SW" V 9150 3350 50  0000 C CNN
-F 2 "prettylib:MX_KAILH_SOCKET_WS2812_1U" H 9400 3650 60  0001 C CNN
+F 2 "prettylib:MX_KAILH_SOCKET_SK9822_1U" H 9400 3650 60  0001 C CNN
 F 3 "" H 9400 3650 60  0000 C CNN
 	2    9400 3650
@@
 	8650 3650 8650 5800
 Connection ~ 9250 3650
+$Comp
+L LED:APA102-2020 D8
+U 1 1 5F71D278
+P 9650 1000
+F 0 "D8" H 9650 1481 50  0000 C CNN
+F 1 "APA102-2020" H 9650 1390 50  0000 C CNN
+F 2 "prettylib:LED-APA102-2020" H 9700 700 50  0001 L TNN
+F 3 "http://www.led-color.com/upload/201604/APA102-2020%20SMD%20LED.pdf" H 9750 625 50  0001 L TNN
+	1    9650 1000
+	1    0    0    -1
+$EndComp
+$Comp
+L LED:APA102-2020 D28
+U 1 1 5F71D76A
+P 10450 1000
+F 0 "D28" H 10450 1481 50  0000 C CNN
+F 1 "APA102-2020" H 10450 1390 50  0000 C CNN
+F 2 "prettylib:LED-APA102-2020" H 10500 700 50  0001 L TNN
+F 3 "http://www.led-color.com/upload/201604/APA102-2020%20SMD%20LED.pdf" H 10550 625 50  0001 L TNN
+	1    10450 1000
+	1    0    0    -1
+$EndComp
+Wire Wire Line
+	9950 900  10150 900
+Wire Wire Line
+	10150 1000 9950 1000
+Wire Wire Line
+	9650 1300 10450 1300
+Wire Wire Line
+	10450 700  10050 700
+$Comp
+L LED:APA102-2020 D33
+U 1 1 5F747BC1
+P 11150 1000
+F 0 "D33" H 11150 1481 50  0000 C CNN
+F 1 "APA102-2020" H 11150 1390 50  0000 C CNN
+F 2 "prettylib:LED-APA102-2020" H 11200 700 50  0001 L TNN
+F 3 "http://www.led-color.com/upload/201604/APA102-2020%20SMD%20LED.pdf" H 11250 625 50  0001 L TNN
+	1    11150 1000
+	1    0    0    -1
+$EndComp
+Wire Wire Line
+	10750 900  10850 900
+Wire Wire Line
+	10850 1000 10750 1000
+Wire Wire Line
+	11150 700  10450 700
+Connection ~ 10450 700
+Wire Wire Line
+	10450 1300 10850 1300
+Connection ~ 10450 1300
+$Comp
+L YAEMK:+5V #PWR0105
+U 1 1 5F772FC4
+P 10050 700
+F 0 "#PWR0105" H 10050 800 30  0001 C CNN
+F 1 "+5V" H 10064 838 30  0000 C CNN
+F 2 "" H 10050 700 60  0000 C CNN
+F 3 "" H 10050 700 60  0000 C CNN
+	1    10050 700
+	1    0    0    -1
+$EndComp
+Connection ~ 10050 700
+Wire Wire Line
+	10050 700  9650 700
+$Comp
+L YAEMK:VSS #PWR0114
+U 1 1 5F773F24
+P 10850 1300
+F 0 "#PWR0114" H 10850 1300 30  0001 C CNN
+F 1 "VSS" H 10850 1359 30  0000 C CNN
+F 2 "" H 10850 1300 60  0000 C CNN
+F 3 "" H 10850 1300 60  0000 C CNN
+	1    10850 1300
+	1    0    0    -1
+$EndComp
+Connection ~ 10850 1300
+Wire Wire Line
+	10850 1300 11150 1300
 $EndSCHEMATC

Commit message: Update YAEMK 1
Parts:
- removed D28, D33, D8: APA102-2020, prettylib:LED-APA102-2020, symbol LED:APA102-2020
Connections:
- wire segments 175 -> 165
Changed lines of the file:
@@
 	8650 3650 8650 5800
 Connection ~ 9250 3650
-$Comp
-L LED:APA102-2020 D8
-U 1 1 5F71D278
-P 9650 1000
-F 0 "D8" H 9650 1481 50  0000 C CNN
-F 1 "APA102-2020" H 9650 1390 50  0000 C CNN
-F 2 "prettylib:LED-APA102-2020" H 9700 700 50  0001 L TNN
-F 3 "http://www.led-color.com/upload/201604/APA102-2020%20SMD%20LED.pdf" H 9750 625 50  0001 L TNN
-	1    9650 1000
-	1    0    0    -1
-$EndComp
-$Comp
-L LED:APA102-2020 D28
-U 1 1 5F71D76A
-P 10450 1000
-F 0 "D28" H 10450 1481 50  0000 C CNN
-F 1 "APA102-2020" H 10450 1390 50  0000 C CNN
-F 2 "prettylib:LED-APA102-2020" H 10500 700 50  0001 L TNN
-F 3 "http://www.led-color.com/upload/201604/APA102-2020%20SMD%20LED.pdf" H 10550 625 50  0001 L TNN
-	1    10450 1000
-	1    0    0    -1
-$EndComp
-Wire Wire Line
-	9950 900  10150 900
-Wire Wire Line
-	10150 1000 9950 1000
-Wire Wire Line
-	9650 1300 10450 1300
-Wire Wire Line
-	10450 700  10050 700
-$Comp
-L LED:APA102-2020 D33
-U 1 1 5F747BC1
-P 11150 1000
-F 0 "D33" H 11150 1481 50  0000 C CNN
-F 1 "APA102-2020" H 11150 1390 50  0000 C CNN
-F 2 "prettylib:LED-APA102-2020" H 11200 700 50  0001 L TNN
-F 3 "http://www.led-color.com/upload/201604/APA102-2020%20SMD%20LED.pdf" H 11250 625 50  0001 L TNN
-	1    11150 1000
-	1    0    0    -1
-$EndComp
-Wire Wire Line
-	10750 900  10850 900
-Wire Wire Line
-	10850 1000 10750 1000
-Wire Wire Line
-	11150 700  10450 700
-Connection ~ 10450 700
-Wire Wire Line
-	10450 1300 10850 1300
-Connection ~ 10450 1300
-$Comp
-L YAEMK:+5V #PWR0105
-U 1 1 5F772FC4
-P 10050 700
-F 0 "#PWR0105" H 10050 800 30  0001 C CNN
-F 1 "+5V" H 10064 838 30  0000 C CNN
-F 2 "" H 10050 700 60  0000 C CNN
-F 3 "" H 10050 700 60  0000 C CNN
-	1    10050 700
-	1    0    0    -1
-$EndComp
-Connection ~ 10050 700
-Wire Wire Line
-	10050 700  9650 700
-$Comp
-L YAEMK:VSS #PWR0114
-U 1 1 5F773F24
-P 10850 1300
-F 0 "#PWR0114" H 10850 1300 30  0001 C CNN
-F 1 "VSS" H 10850 1359 30  0000 C CNN
-F 2 "" H 10850 1300 60  0000 C CNN
-F 3 "" H 10850 1300 60  0000 C CNN
-	1    10850 1300
-	1    0    0    -1
-$EndComp
-Connection ~ 10850 1300
-Wire Wire Line
-	10850 1300 11150 1300
 $EndSCHEMATC

Commit message: Sync
Connections:
- net labels added: VDD
- net labels removed: +5V
Changed lines of the file:
@@
 Connection ~ 9250 2150
-$Comp
-L YAEMK:+5V #PWR09
-U 1 1 5ECF0880
-P 5350 1600
-F 0 "#PWR09" H 5350 1700 30  0001 C CNN
-F 1 "+5V" H 5364 1738 30  0000 C CNN
-F 2 "" H 5350 1600 60  0000 C CNN
-F 3 "" H 5350 1600 60  0000 C CNN
-	1    5350 1600
-	1    0    0    -1
-$EndComp
 $Comp
 L YAEMK:VSS #PWR08
@@
 	8650 3650 8650 5800
 Connection ~ 9250 3650
+$Comp
+L YAEMK:VDD #PWR0105
+U 1 1 5FB0F6DB
+P 5350 1600
+F 0 "#PWR0105" H 5350 1700 30  0001 C CNN
+F 1 "VDD" H 5364 1738 30  0000 C CNN
+F 2 "" H 5350 1600 60  0000 C CNN
+F 3 "" H 5350 1600 60  0000 C CNN
+	1    5350 1600
+	1    0    0    -1
+$EndComp
 $EndSCHEMATC

Commit message: One step further
Parts:
- added C48, C49, C50, C51, C52, C53: 100n, prettylib:SMD-0603, symbol YAEMK:C
- added D71, D72, D73, D74, D75, D76: SW, prettylib:SK6812_mini_e_flippable, symbol YAEMK:SK6812MINI-E
- D35, D38: renamed from S5; footprint prettylib:MX_KAILH_SOCKET_WS2812_2U_2X1U -> prettylib:SK6812_mini_e_flippable; symbol YAEMK:MX_WS2812_2U_2X1U -> YAEMK:SK6812MINI-E
- D36: renamed from S1; footprint prettylib:MX_KAILH_SOCKET_WS2812_2U_2X1U -> prettylib:SK6812_mini_flipable; symbol YAEMK:MX_WS2812_2U_2X1U -> YAEMK:SK6812MINI
- D37: renamed from S1; footprint prettylib:MX_KAILH_SOCKET_WS2812_2U_2X1U -> prettylib:SK6812_mini_e_flippable; symbol YAEMK:MX_WS2812_2U_2X1U -> YAEMK:SK6812MINI-E
- D39: renamed from S13; footprint prettylib:MX_KAILH_SOCKET_SK9822_1U -> prettylib:SK6812_mini_e_flippable; symbol YAEMK:MX_WS2812_1U -> YAEMK:SK6812MINI-E
- D40: renamed from S18; footprint prettylib:MX_KAILH_SOCKET_SK9822_1U -> prettylib:SK6812_mini_e_flippable; symbol YAEMK:MX_WS2812_1U -> YAEMK:SK6812MINI-E
- D41: renamed from S35; footprint prettylib:MX_KAILH_SOCKET_SK9822_1U -> prettylib:SK6812_mini_flipable; symbol YAEMK:MX_WS2812_1U -> YAEMK:SK6812MINI
- D42: renamed from S34; footprint prettylib:MX_KAILH_SOCKET_SK9822_1U -> prettylib:SK6812_mini_e_flippable; symbol YAEMK:MX_WS2812_1U -> YAEMK:SK6812MINI-E
- D43: renamed from S33; footprint prettylib:MX_KAILH_SOCKET_SK9822_1U -> prettylib:SK6812_mini_flipable; symbol YAEMK:MX_WS2812_1U -> YAEMK:SK6812MINI
- D44: renamed from S32; footprint prettylib:MX_KAILH_SOCKET_SK9822_1U -> prettylib:SK6812_mini_e_flippable; symbol YAEMK:MX_WS2812_1U -> YAEMK:SK6812MINI-E
- D45: renamed from S28; footprint prettylib:MX_KAILH_SOCKET_SK9822_1U -> prettylib:SK6812_mini_e_flippable; symbol YAEMK:MX_WS2812_1U -> YAEMK:SK6812MINI-E
- D46: renamed from S29; footprint prettylib:MX_KAILH_SOCKET_SK9822_1U -> prettylib:SK6812_mini_e_flippable; symbol YAEMK:MX_WS2812_1U -> YAEMK:SK6812MINI-E
- D47: renamed from S30; footprint prettylib:MX_KAILH_SOCKET_SK9822_1U -> prettylib:SK6812_mini_e_flippable; symbol YAEMK:MX_WS2812_1U -> YAEMK:SK6812MINI-E
- D48: renamed from S31; footprint prettylib:MX_KAILH_SOCKET_SK9822_1U -> prettylib:SK6812_mini_e_flippable; symbol YAEMK:MX_WS2812_1U -> YAEMK:SK6812MINI-E
- D49: renamed from S27; footprint prettylib:MX_KAILH_SOCKET_SK9822_1U -> prettylib:SK6812_mini_e_flippable; symbol YAEMK:MX_WS2812_1U -> YAEMK:SK6812MINI-E
- D50: renamed from S26; footprint prettylib:MX_KAILH_SOCKET_SK9822_1U -> prettylib:SK6812_mini_e_flippable; symbol YAEMK:MX_WS2812_1U -> YAEMK:SK6812MINI-E
- D51: renamed from S25; footprint prettylib:MX_KAILH_SOCKET_SK9822_1U -> prettylib:SK6812_mini_e_flippable; symbol YAEMK:MX_WS2812_1U -> YAEMK:SK6812MINI-E
- D52: renamed from S24; footprint prettylib:MX_KAILH_SOCKET_SK9822_1U -> prettylib:SK6812_mini_e_flippable; symbol YAEMK:MX_WS2812_1U -> YAEMK:SK6812MINI-E
- D53: renamed from S19; footprint prettylib:MX_KAILH_SOCKET_SK9822_1U -> prettylib:SK6812_mini_e_flippable; symbol YAEMK:MX_WS2812_1U -> YAEMK:SK6812MINI-E
- D54: renamed from S20; footprint prettylib:MX_KAILH_SOCKET_SK9822_1U -> prettylib:SK6812_mini_e_flippable; symbol YAEMK:MX_WS2812_1U -> YAEMK:SK6812MINI-E
- D55: renamed from S21; footprint prettylib:MX_KAILH_SOCKET_SK9822_1U -> prettylib:SK6812_mini_e_flippable; symbol YAEMK:MX_WS2812_1U -> YAEMK:SK6812MINI-E
- D56: renamed from S22; footprint prettylib:MX_KAILH_SOCKET_SK9822_1U -> prettylib:SK6812_mini_e_flippable; symbol YAEMK:MX_WS2812_1U -> YAEMK:SK6812MINI-E
- D57: renamed from S17; footprint prettylib:MX_KAILH_SOCKET_SK9822_1U -> prettylib:SK6812_mini_e_flippable; symbol YAEMK:MX_WS2812_1U -> YAEMK:SK6812MINI-E
- D58: renamed from S16; footprint prettylib:MX_KAILH_SOCKET_SK9822_1U -> prettylib:SK6812_mini_e_flippable; symbol YAEMK:MX_WS2812_1U -> YAEMK:SK6812MINI-E
- D59: renamed from S15; footprint prettylib:MX_KAILH_SOCKET_SK9822_1U -> prettylib:SK6812_mini_flipable; symbol YAEMK:MX_WS2812_1U -> YAEMK:SK6812MINI
- D60: renamed from S14; footprint prettylib:MX_KAILH_SOCKET_SK9822_1U -> prettylib:SK6812_mini_e_flippable; symbol YAEMK:MX_WS2812_1U -> YAEMK:SK6812MINI-E
- D61: renamed from S9; footprint prettylib:MX_KAILH_SOCKET_SK9822_1U -> prettylib:SK6812_mini_e_flippable; symbol YAEMK:MX_WS2812_1U -> YAEMK:SK6812MINI-E
- D62: renamed from S10; footprint prettylib:MX_KAILH_SOCKET_SK9822_1U -> prettylib:SK6812_mini_flipable; symbol YAEMK:MX_WS2812_1U -> YAEMK:SK6812MINI
- D63: renamed from S11; footprint prettylib:MX_KAILH_SOCKET_SK9822_1U -> prettylib:SK6812_mini_e_flippable; symbol YAEMK:MX_WS2812_1U -> YAEMK:SK6812MINI-E
- D64: renamed from S12; footprint prettylib:MX_KAILH_SOCKET_SK9822_1U -> prettylib:SK6812_mini_e_flippable; symbol YAEMK:MX_WS2812_1U -> YAEMK:SK6812MINI-E
- D65: renamed from S4; footprint prettylib:MX_KAILH_SOCKET_SK9822_1U -> prettylib:SK6812_mini_flipable; symbol YAEMK:MX_WS2812_1U -> YAEMK:SK6812MINI
- D66: renamed from S3; footprint prettylib:MX_KAILH_SOCKET_SK9822_1U -> prettylib:SK6812_mini_e_flippable; symbol YAEMK:MX_WS2812_1U -> YAEMK:SK6812MINI-E
- D67: renamed from S2; footprint prettylib:MX_KAILH_SOCKET_SK9822_1U -> prettylib:SK6812_mini_e_flippable; symbol YAEMK:MX_WS2812_1U -> YAEMK:SK6812MINI-E
- renumbered C18 to C11, C14 to C12, C21 to C13, C12 to C14, C20 to C15, C17 to C16, C23 to C17, C19 to C18, C13 to C19, C22 to C20, C24 to C21, C16 to C22, C25 to C23, C15 to C24, C26 to C25, C30 to C26, C4 to C3, C33 to C30, C35 to C31, C31 to C32, C32 to C33, C36 to C35, C5 to C4, C6 to C5, C7 to C6, C8 to C7, C9 to C8, C11 to C9
Connections:
- net TIM2_CH3: now also D35.4 (DIN); no longer D35.3 (DIN)
- net VDD: now also C10.1, C11.1, C12.1, C13.1, C14.1, C15.1, C16.1, C17.1, C18.1, C19.1, C20.1, C21.1, C22.1, C23.1, C24.1, C25.1, C26.1, C27.1, C28.1, C29.1, C3.1, C30.1, C31.1, C32.1, C33.1, C34.1, C35.1, C4.1, C5.1, C6.1, C7.1, C8.1, C9.1, D35.1 (VDD), D37.1 (VDD), D38.1 (VDD), D39.1 (VDD), D40.1 (VDD), D42.1 (VDD), D44.1 (VDD), D45.1 (VDD), D46.1 (VDD), D47.1 (VDD), D48.1 (VDD), D49.1 (VDD), D50.1 (VDD), D51.1 (VDD), D52.1 (VDD), D53.1 (VDD), D54.1 (VDD), D55.1 (VDD), D56.1 (VDD), D57.1 (VDD), D58.1 (VDD), D60.1 (VDD), D61.1 (VDD), D63.1 (VDD), D64.1 (VDD), D66.1 (VDD), D67.1 (VDD), C48.1, C49.1, C50.1, C51.1, C52.1, C53.1, D71.1 (VDD), D72.1 (VDD), D73.1 (VDD), D74.1 (VDD), D75.1 (VDD), D76.1 (VDD); no longer C10.2, C11.2, C12.2, C13.2, C14.2, C15.2, C16.2, C17.2, C18.2, C19.2, C20.2, C21.2, C22.2, C23.2, C24.2, C25.2, C26.2, C27.2, C28.2, C29.2, C3.2, C30.2, C31.2, C32.2, C33.2, C34.2, C35.2, C4.2, C5.2, C6.2, C7.2, C8.2, C9.2, D35.4 (VDD), D37.8 (VDD), D38.8 (VDD), D39.4 (VDD), D40.4 (VDD), D42.4 (VDD), D44.4 (VDD), D45.4 (VDD), D46.4 (VDD), D47.4 (VDD), D48.4 (VDD), D49.4 (VDD), D50.4 (VDD), D51.4 (VDD), D52.4 (VDD), D53.4 (VDD), D54.4 (VDD), D55.4 (VDD), D56.4 (VDD), D57.4 (VDD), D58.4 (VDD), D60.4 (VDD), D61.4 (VDD), D63.4 (VDD), D64.4 (VDD), D66.4 (VDD), D67.4 (VDD)
- net VSS: now also C10.2, C11.2, C12.2, C13.2, C14.2, C15.2, C16.2, C17.2, C18.2, C19.2, C20.2, C21.2, C22.2, C23.2, C24.2, C25.2, C26.2, C27.2, C28.2, C29.2, C3.2, C30.2, C31.2, C32.2, C33.2, C34.2, C35.2, C4.2, C5.2, C6.2, C7.2, C8.2, C9.2, D35.3 (VSS), D37.3 (VSS), D38.3 (VSS), D39.3 (VSS), D40.3 (VSS), D42.3 (VSS), D44.3 (VSS), D45.3 (VSS), D46.3 (VSS), D47.3 (VSS), D48.3 (VSS), D49.3 (VSS), D50.3 (VSS), D51.3 (VSS), D52.3 (VSS), D53.3 (VSS), D54.3 (VSS), D55.3 (VSS), D56.3 (VSS), D57.3 (VSS), D58.3 (VSS), D60.3 (VSS), D61.3 (VSS), D63.3 (VSS), D64.3 (VSS), D66.3 (VSS), D67.3 (VSS), C48.2, C49.2, C50.2, C51.2, C52.2, C53.2, D71.3 (VSS), D72.3 (VSS), D73.3 (VSS), D74.3 (VSS), D75.3 (VSS), D76.3 (VSS); no longer C10.1, C11.1, C12.1, C13.1, C14.1, C15.1, C16.1, C17.1, C18.1, C19.1, C20.1, C21.1, C22.1, C23.1, C24.1, C25.1, C26.1, C27.1, C28.1, C29.1, C3.1, C30.1, C31.1, C32.1, C33.1, C34.1, C35.1, C4.1, C5.1, C6.1, C7.1, C8.1, C9.1, D35.2 (VSS), D37.6 (VSS), D38.6 (VSS), D39.2 (VSS), D40.2 (VSS), D42.2 (VSS), D44.2 (VSS), D45.2 (VSS), D46.2 (VSS), D47.2 (VSS), D48.2 (VSS), D49.2 (VSS), D50.2 (VSS), D51.2 (VSS), D52.2 (VSS), D53.2 (VSS), D54.2 (VSS), D55.2 (VSS), D56.2 (VSS), D57.2 (VSS), D58.2 (VSS), D60.2 (VSS), D61.2 (VSS), D63.2 (VSS), D64.2 (VSS), D66.2 (VSS), D67.2 (VSS)
- net at D36.3 (DIN): now also D35.2 (DOUT); no longer D35.1 (DOUT)
- net at D41.3 (DIN): now also D42.2 (DOUT); no longer D40.1 (DOUT)
- net at D59.1 (DOUT): now also D60.4 (DIN); no longer D60.3 (DIN)
- net at D65.1 (DOUT): now also D67.4 (DIN); no longer D66.3 (DIN)
- net at D36.1 (DOUT): now also D37.4 (DIN); no longer D37.7 (DIN)
- net at D41.1 (DOUT): now also D46.4 (DIN); no longer D42.3 (DIN)
- net at D62.3 (DIN): now also D61.2 (DOUT); no longer D61.1 (DOUT)
- net at D43.3 (DIN): now also D44.2 (DOUT); no longer D42.1 (DOUT)
- net at D62.1 (DOUT): now also D63.4 (DIN); no longer D63.3 (DIN)
- net at D43.1 (DOUT): now also D45.4 (DIN); no longer D44.3 (DIN)
- net at D59.3 (DIN): now also D58.2 (DOUT); no longer D58.1 (DOUT)
- net at D65.3 (DIN): now also D66.2 (DOUT); no longer D64.1 (DOUT)
- new net: D40.2 (DOUT), D42.4 (DIN)
- new net: D39.2 (DOUT), D40.4 (DIN)
- new net: D45.2 (DOUT), D47.4 (DIN)
- new net: D50.2 (DOUT), D51.4 (DIN)
- new net: D49.2 (DOUT), D50.4 (DIN)
- new net: D55.2 (DOUT), D56.4 (DIN)
- new net: D54.2 (DOUT), D55.4 (DIN)
- new net: D60.2 (DOUT), D61.4 (DIN)
- new net: D64.2 (DOUT), D66.4 (DIN)
- new net: D44.4 (DIN), D46.2 (DOUT)
- new net: D51.2 (DOUT), D52.4 (DIN)
- new net: D56.2 (DOUT), D57.4 (DIN)
- new net: D37.2 (DOUT), D38.4 (DIN)
- new net: D47.2 (DOUT), D48.4 (DIN)
- new net: D52.2 (DOUT), D53.4 (DIN)
- new net: D57.2 (DOUT), D58.4 (DIN)
- new net: D38.2 (DOUT), D39.4 (DIN)
- new net: D48.2 (DOUT), D49.4 (DIN)
- new net: D53.2 (DOUT), D54.4 (DIN)
- new net: D63.2 (DOUT), D64.4 (DIN)
- new net: D67.2 (DOUT), D71.4 (DIN)
- new net: D75.2 (DOUT), D76.4 (DIN)
- new net: D74.2 (DOUT), D75.4 (DIN)
- new net: D73.2 (DOUT), D74.4 (DIN)
- new net: D72.2 (DOUT), D73.4 (DIN)
- new net: D71.2 (DOUT), D72.4 (DIN)
Other:
- moved on the sheet: C10, C11, C12, C13, C14, C15, C16, C17, C18, C19, C20, C21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

Commit message: RC
Parts:
- added JP3, JP4, JP5, JP6, JP7, JP8: SolderJumper_2_Open, prettylib:SOLDER_JUMPER_2, symbol Jumper:SolderJumper_2_Open
Connections:
- net at D35.2 (DOUT), D36.3 (DIN): now also JP3.1 (A)
- net at D43.1 (DOUT), D45.4 (DIN): now also JP8.2 (B)
- net at D59.1 (DOUT), D60.4 (DIN): now also JP7.1 (A)
- net at D65.3 (DIN), D66.2 (DOUT): now also JP4.2 (B)
- net at D36.1 (DOUT), D37.4 (DIN): now also JP3.2 (B)
- net at D41.1 (DOUT), D46.4 (DIN): now also JP6.2 (B)
- net at D41.3 (DIN), D42.2 (DOUT): now also JP6.1 (A)
- net at D61.2 (DOUT), D62.3 (DIN): now also JP5.2 (B)
- net at D62.1 (DOUT), D63.4 (DIN): now also JP5.1 (A)
- net at D43.3 (DIN), D44.2 (DOUT): now also JP8.1 (A)
- net at D58.2 (DOUT), D59.3 (DIN): now also JP7.2 (B)
- net at D65.1 (DOUT), D67.4 (DIN): now also JP4.1 (A)
Changed lines of the file:
@@
 Wire Wire Line
 	11000 4800 10950 4800
+$Comp
+L Jumper:SolderJumper_2_Open JP3
+U 1 1 5FC59A5F
+P 1700 3250
+F 0 "JP3" H 1700 3455 50  0000 C CNN
+F 1 "SolderJumper_2_Open" H 1700 3364 50  0000 C CNN
+F 2 "prettylib:SOLDER_JUMPER_2" H 1700 3250 50  0001 C CNN
+F 3 "~" H 1700 3250 50  0001 C CNN
+	1    1700 3250
+	1    0    0    -1
+$EndComp
+$Comp
+L Jumper:SolderJumper_2_Open JP4
+U 1 1 5FC5EAF9
+P 2250 5300
+F 0 "JP4" H 2250 5505 50  0000 C CNN
+F 1 "SolderJumper_2_Open" H 2250 5414 50  0000 C CNN
+F 2 "prettylib:SOLDER_JUMPER_2" H 2250 5300 50  0001 C CNN
+F 3 "~" H 2250 5300 50  0001 C CNN
+	1    2250 5300
+	1    0    0    -1
+$EndComp
+$Comp
+L Jumper:SolderJumper_2_Open JP5
+U 1 1 5FC601CD
+P 4650 5300
+F 0 "JP5" H 4650 5505 50  0000 C CNN
+F 1 "SolderJumper_2_Open" H 4650 5414 50  0000 C CNN
+F 2 "prettylib:SOLDER_JUMPER_2" H 4650 5300 50  0001 C CNN
+F 3 "~" H 4650 5300 50  0001 C CNN
+	1    4650 5300
+	1    0    0    -1
+$EndComp
+$Comp
+L Jumper:SolderJumper_2_Open JP7
+U 1 1 5FC6267C
+P 6450 5300
+F 0 "JP7" H 6450 5505 50  0000 C CNN
+F 1 "SolderJumper_2_Open" H 6450 5414 50  0000 C CNN
+F 2 "prettylib:SOLDER_JUMPER_2" H 6450 5300 50  0001 C CNN
+F 3 "~" H 6450 5300 50  0001 C CNN
+	1    6450 5300
+	1    0    0    -1
+$EndComp
+$Comp
+L Jumper:SolderJumper_2_Open JP8
+U 1 1 5FC68D55
+P 7100 3300
+F 0 "JP8" H 7100 3505 50  0000 C CNN
+F 1 "SolderJumper_2_Open" H 7100 3414 50  0000 C CNN
+F 2 "prettylib:SOLDER_JUMPER_2" H 7100 3300 50  0001 C CNN
+F 3 "~" H 7100 3300 50  0001 C CNN
+	1    7100 3300
+	1    0    0    -1
+$EndComp
+$Comp
+L Jumper:SolderJumper_2_Open JP6
+U 1 1 5FC6B932
+P 5300 3300
+F 0 "JP6" H 5300 3505 50  0000 C CNN
+F 1 "SolderJumper_2_Open" H 5300 3414 50  0000 C CNN
+F 2 "prettylib:SOLDER_JUMPER_2" H 5300 3300 50  0001 C CNN
+F 3 "~" H 5300 3300 50  0001 C CNN
+	1    5300 3300
+	1    0    0    -1
+$EndComp
+Wire Wire Line
+	5000 3800 5000 3300
+Wire Wire Line
+	5000 3300 5150 3300
+Connection ~ 5000 3800
+Wire Wire Line
+	5450 3300 5600 3300
+Wire Wire Line
+	5600 3300 5600 3800
+Connection ~ 5600 3800
+Wire Wire Line
+	1850 3250 2000 3250
+Wire Wire Line
+	2000 3250 2000 3800
+Connection ~ 2000 3800
+Wire Wire Line
+	1550 3250 1400 3250
+Wire Wire Line
+	1400 3250 1400 3800
+Connection ~ 1400 3800
+Wire Wire Line
+	6800 3800 6800 3300
+Wire Wire Line
+	6800 3300 6950 3300
+Connection ~ 6800 3800
+Wire Wire Line
+	7250 3300 7400 3300
+Wire Wire Line
+	7400 3300 7400 3800
+Connection ~ 7400 3800
+Wire Wire Line
+	6600 5300 6750 5300
+Wire Wire Line
+	6750 5300 6750 4800
+Connection ~ 6750 4800
+Wire Wire Line
+	6150 4800 6150 5300
+Wire Wire Line
+	6150 5300 6300 5300
+Connection ~ 6150 4800
+Wire Wire Line
+	4800 5300 4950 5300
+Wire Wire Line
+	4950 5300 4950 4800
+Connection ~ 4950 4800
+Wire Wire Line
+	4350 4800 4350 5300
+Wire Wire Line
+	4350 5300 4500 5300
+Connection ~ 4350 4800
+Wire Wire Line
+	2550 4800 2550 5300
+Wire Wire Line
+	2550 5300 2400 5300
+Connection ~ 2550 4800
+Wire Wire Line
+	1950 4800 1950 5300
+Wire Wire Line
+	1950 5300 2100 5300
+Connection ~ 1950 4800
 $EndSCHEMATC
