File: PCB/mcu.sch (KiCad schematic (older format))
At the start: 54 parts, among them J1 DBG, P1 PC, P2 Link, P3 SSD1107, Q1 Q_PNP_BCE, U1 24LC64, U2 TLV62568DBV, U3 USBLC6-2SC6, U4 USBLC6-2SC6, U5 STM32F303CCTx

Commit message: YAEMK 1.2 RC
Parts:
- removed Q1: Q_PNP_BCE, prettylib:SOT-23, symbol Device:Q_PNP_BCE
- added C54: 100n, prettylib:SMD-0603, symbol YAEMK:C
- added F1: 3A, prettylib:Fuse_1206_3216Metric, symbol Device:Polyfuse_Small
- added F2: 1.5A, prettylib:Fuse_1206_3216Metric, symbol Device:Polyfuse_Small
- added JP10: +3V3, prettylib:SOLDER_JUMPER_2, symbol YAEMK-rescue:SolderJumper_2_Open-YAEMK
- added JP9: +5V, prettylib:SOLDER_JUMPER_2, symbol YAEMK-rescue:SolderJumper_2_Open-YAEMK
- added Q1: MMUN2133LT1G, prettylib:SOT-23, symbol Device:Q_PNP_BEC_BRT
- D68, D69: value DIODE -> 1N4148; footprint Diode_SMD:D_SOD-523 -> prettylib:D_SOD-523
- D77: footprint Diode_SMD:D_SOD-123F -> prettylib:D_SOD-323_HandSoldering
- HSE1: footprint Crystal:Crystal_SMD_3225-4Pin_3.2x2.5mm -> prettylib:Crystal_SMD_3225-4Pin_3.2x2.5mm
- L1: footprint Inductor_SMD:L_Taiyo-Yuden_MD-3030 -> prettylib:L_Taiyo-Yuden_MD-3030
- R11: value 120R -> 120
- R15: value 1k5 -> 450k
- R16, R23: value 1k5 -> 100k
- R22, R26: value 1k5 -> 5k1
- R24, R25: value 1k5 -> 10k
- U1: footprint Package_SO:TSSOP-8_4.4x3mm_P0.65mm -> prettylib:TSSOP-8_4.4x3mm_P0.65mm
- U2: value TLV62568DBV -> TLV62568DBVR; footprint Package_TO_SOT_SMD:SOT-23-5 -> prettylib:SOT-23-5
Connections:
- net labels added: PLUG_DETECT, RGB_VDD, USB_VBUS_IN_FUSED
- net labels removed: SPLIT_DETECT
- wire segments 170 -> 185
- no-connect marks 9 -> 12
Other:
- note added: "Fuses and plug detect"
- note added: "Input Voltage Regulator"
- note added: "RGB Led supply voltage selection"
- note added: "SWD / JTAG Interface\n"
- note removed: "Input Voltage Regulator MCU"
- note removed: "JTAG Interface\n"
- moved on the sheet: C36, C37, C38, C39, C40, C41, C42, D68, D69, D77, J1, P3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

Commit message: Clean up save point
Parts:
- removed JP10: +3V3, prettylib:SOLDER_JUMPER_2, symbol YAEMK-rescue:SolderJumper_2_Open-YAEMK
- removed JP9: +5V, prettylib:SOLDER_JUMPER_2, symbol YAEMK-rescue:SolderJumper_2_Open-YAEMK
- D70: footprint prettylib:LED-0603 -> prettylib:LED-0603_flipable
- S32, S33: footprint prettylib:SMD_Tacticle_Switch_TS24CA -> prettylib:SMD_Tacticle_Switch_TS24CA_flipable
Other:
- note removed: "RGB Led supply voltage selection"
