File: PCB/YAEMK.sch (KiCad schematic (older format))
At the start: 81 parts, among them SW1 ALPS EC11

Commit message: Add WIP yaemk 1.2 files
Parts:
- S10, S11, S12, S13, S14, S15, S16, S17, S18, S19, S2, S20, S21, S22, S24, S25, S26, S27, S28, S29, S3, S30, S31, S32, S33, S34, S35, S4, S9: footprint prettylib:MX_KAILH_SOCKET_WS2812_1U -> prettylib:MX_KAILH_SOCKET_SK9822_1U
Changed lines of the file:
@@
 F 0 "S2" H 1600 50  60  0000 C CNN
 F 1 "SW" H 1600 -100 60  0000 C CNN
-F 2 "prettylib:MX_KAILH_SOCKET_WS2812_1U" H 1600 400 60  0001 C CNN
+F 2 "prettylib:MX_KAILH_SOCKET_SK9822_1U" H 1600 400 60  0001 C CNN
 F 3 "~" H 1600 400 60  0000 C CNN
 	1    1600 400
@@
 F 0 "S9" H 2300 50  60  0000 C CNN
 F 1 "SW" H 2300 -100 60  0000 C CNN
-F 2 "prettylib:MX_KAILH_SOCKET_WS2812_1U" H 2300 400 60  0001 C CNN
+F 2 "prettylib:MX_KAILH_SOCKET_SK9822_1U" H 2300 400 60  0001 C CNN
 F 3 "~" H 2300 400 60  0000 C CNN
 	1    2300 400
@@
 F 0 "S14" H 3000 50  60  0000 C CNN
 F 1 "SW" H 3000 -100 60  0000 C CNN
-F 2 "prettylib:MX_KAILH_SOCKET_WS2812_1U" H 3000 400 60  0001 C CNN
+F 2 "prettylib:MX_KAILH_SOCKET_SK9822_1U" H 3000 400 60  0001 C CNN
 F 3 "~" H 3000 400 60  0000 C CNN
 	1    3000 400
@@
 F 0 "S19" H 3700 50  60  0000 C CNN
 F 1 "SW" H 3700 -100 60  0000 C CNN
-F 2 "prettylib:MX_KAILH_SOCKET_WS2812_1U" H 3700 400 60  0001 C CNN
+F 2 "prettylib:MX_KAILH_SOCKET_SK9822_1U" H 3700 400 60  0001 C CNN
 F 3 "~" H 3700 400 60  0000 C CNN
 	1    3700 400
@@
 F 0 "S24" H 4400 50  60  0000 C CNN
 F 1 "SW" H 4400 -100 60  0000 C CNN
-F 2 "prettylib:MX_KAILH_SOCKET_WS2812_1U" H 4400 400 60  0001 C CNN
+F 2 "prettylib:MX_KAILH_SOCKET_SK9822_1U" H 4400 400 60  0001 C CNN
 F 3 "~" H 4400 400 60  0000 C CNN
 	1    4400 400
@@
 F 0 "S28" H 5100 50  60  0000 C CNN
 F 1 "SW" H 5100 -100 60  0000 C CNN
-F 2 "prettylib:MX_KAILH_SOCKET_WS2812_1U" H 5100 400 60  0001 C CNN
+F 2 "prettylib:MX_KAILH_SOCKET_SK9822_1U" H 5100 400 60  0001 C CNN
 F 3 "~" H 5100 400 60  0000 C CNN
 	1    5100 400
@@
 F 0 "S32" H 5800 50  60  0000 C CNN
 F 1 "SW" H 5800 -100 60  0000 C CNN
-F 2 "prettylib:MX_KAILH_SOCKET_WS2812_1U" H 5800 400 60  0001 C CNN
+F 2 "prettylib:MX_KAILH_SOCKET_SK9822_1U" H 5800 400 60  0001 C CNN
 F 3 "~" H 5800 400 60  0000 C CNN
 	1    5800 400
@@
 F 0 "S3" H 1600 750 60  0000 C CNN
 F 1 "SW" H 1600 600 60  0000 C CNN
-F 2 "prettylib:MX_KAILH_SOCKET_WS2812_1U" H 1600 1100 60  0001 C CNN
+F 2 "prettylib:MX_KAILH_SOCKET_SK9822_1U" H 1600 1100 60  0001 C CNN
 F 3 "~" H 1600 1100 60  0000 C CNN
 	1    1600 1100
@@
 F 0 "S10" H 2300 750 60  0000 C CNN
 F 1 "SW" H 2300 600 60  0000 C CNN
-F 2 "prettylib:MX_KAILH_SOCKET_WS2812_1U" H 2300 1100 60  0001 C CNN
+F 2 "prettylib:MX_KAILH_SOCKET_SK9822_1U" H 2300 1100 60  0001 C CNN
 F 3 "~" H 2300 1100 60  0000 C CNN
 	1    2300 1100
@@
 F 0 "S15" H 3000 750 60  0000 C CNN
 F 1 "SW" H 3000 600 60  0000 C CNN
-F 2 "prettylib:MX_KAILH_SOCKET_WS2812_1U" H 3000 1100 60  0001 C CNN
+F 2 "prettylib:MX_KAILH_SOCKET_SK9822_1U" H 3000 1100 60  0001 C CNN
 F 3 "~" H 3000 1100 60  0000 C CNN
 	1    3000 1100
@@
 F 0 "S20" H 3700 750 60  0000 C CNN
 F 1 "SW" H 3700 600 60  0000 C CNN
-F 2 "prettylib:MX_KAILH_SOCKET_WS2812_1U" H 3700 1100 60  0001 C CNN
+F 2 "prettylib:MX_KAILH_SOCKET_SK9822_1U" H 3700 1100 60  0001 C CNN
 F 3 "~" H 3700 1100 60  0000 C CNN
 	1    3700 1100
@@
 F 0 "S25" H 4400 750 60  0000 C CNN
 F 1 "SW" H 4400 600 60  0000 C CNN
-F 2 "prettylib:MX_KAILH_SOCKET_WS2812_1U" H 4400 1100 60  0001 C CNN
+F 2 "prettylib:MX_KAILH_SOCKET_SK9822_1U" H 4400 1100 60  0001 C CNN
 F 3 "~" H 4400 1100 60  0000 C CNN
 	1    4400 1100
@@
 F 0 "S29" H 5100 750 60  0000 C CNN
 F 1 "SW" H 5100 600 60  0000 C CNN
-F 2 "prettylib:MX_KAILH_SOCKET_WS2812_1U" H 5100 1100 60  0001 C CNN
+F 2 "prettylib:MX_KAILH_SOCKET_SK9822_1U" H 5100 1100 60  0001 C CNN
 F 3 "~" H 5100 1100 60  0000 C CNN
 	1    5100 1100
@@
 F 0 "S11" H 2300 1450 60  0000 C CNN
 F 1 "SW" H 2300 1300 60  0000 C CNN
-F 2 "prettylib:MX_KAILH_SOCKET_WS2812_1U" H 2300 1800 60  0001 C CNN
+F 2 "prettylib:MX_KAILH_SOCKET_SK9822_1U" H 2300 1800 60  0001 C CNN
 F 3 "~" H 2300 1800 60  0000 C CNN
 	1    2300 1800
@@
 F 0 "S16" H 3000 1450 60  0000 C CNN
 F 1 "SW" H 3000 1300 60  0000 C CNN
-F 2 "prettylib:MX_KAILH_SOCKET_WS2812_1U" H 3000 1800 60  0001 C CNN
+F 2 "prettylib:MX_KAILH_SOCKET_SK9822_1U" H 3000 1800 60  0001 C CNN
 F 3 "~" H 3000 1800 60  0000 C CNN
 	1    3000 1800
@@
 F 0 "S21" H 3700 1450 60  0000 C CNN
 F 1 "SW" H 3700 1300 60  0000 C CNN
-F 2 "prettylib:MX_KAILH_SOCKET_WS2812_1U" H 3700 1800 60  0001 C CNN
+F 2 "prettylib:MX_KAILH_SOCKET_SK9822_1U" H 3700 1800 60  0001 C CNN
 F 3 "~" H 3700 1800 60  0000 C CNN
 	1    3700 1800
@@
 F 0 "S26" H 4400 1450 60  0000 C CNN
 F 1 "SW" H 4400 1300 60  0000 C CNN
-F 2 "prettylib:MX_KAILH_SOCKET_WS2812_1U" H 4400 1800 60  0001 C CNN
+F 2 "prettylib:MX_KAILH_SOCKET_SK9822_1U" H 4400 1800 60  0001 C CNN
 F 3 "~" H 4400 1800 60  0000 C CNN
 	1    4400 1800
@@
 F 0 "S30" H 5100 1450 60  0000 C CNN
 F 1 "SW" H 5100 1300 60  0000 C CNN
-F 2 "prettylib:MX_KAILH_SOCKET_WS2812_1U" H 5100 1800 60  0001 C CNN
+F 2 "prettylib:MX_KAILH_SOCKET_SK9822_1U" H 5100 1800 60  0001 C CNN
 F 3 "~" H 5100 1800 60  0000 C CNN
 	1    5100 1800
@@
 F 0 "S34" H 5800 1450 60  0000 C CNN
 F 1 "SW" H 5800 1300 60  0000 C CNN
-F 2 "prettylib:MX_KAILH_SOCKET_WS2812_1U" H 5800 1800 60  0001 C CNN
+F 2 "prettylib:MX_KAILH_SOCKET_SK9822_1U" H 5800 1800 60  0001 C CNN
 F 3 "~" H 5800 1800 60  0000 C CNN
 	1    5800 1800
@@
 F 0 "S12" H 2300 2150 60  0000 C CNN
 F 1 "SW" H 2300 2000 60  0000 C CNN
-F 2 "prettylib:MX_KAILH_SOCKET_WS2812_1U" H 2300 2500 60  0001 C CNN
+F 2 "prettylib:MX_KAILH_SOCKET_SK9822_1U" H 2300 2500 60  0001 C CNN
 F 3 "~" H 2300 2500 60  0000 C CNN
 	1    2300 2500
@@
 F 0 "S17" H 3000 2150 60  0000 C CNN
 F 1 "SW" H 3000 2000 60  0000 C CNN
-F 2 "prettylib:MX_KAILH_SOCKET_WS2812_1U" H 3000 2500 60  0001 C CNN
+F 2 "prettylib:MX_KAILH_SOCKET_SK9822_1U" H 3000 2500 60  0001 C CNN
 F 3 "~" H 3000 2500 60  0000 C CNN
 	1    3000 2500
@@
 F 0 "S22" H 3700 2150 60  0000 C CNN
 F 1 "SW" H 3700 2000 60  0000 C CNN
-F 2 "prettylib:MX_KAILH_SOCKET_WS2812_1U" H 3700 2500 60  0001 C CNN
+F 2 "prettylib:MX_KAILH_SOCKET_SK9822_1U" H 3700 2500 60  0001 C CNN
 F 3 "~" H 3700 2500 60  0000 C CNN
 	1    3700 2500
@@
 F 0 "S27" H 4400 2150 60  0000 C CNN
 F 1 "SW" H 4400 2000 60  0000 C CNN
-F 2 "prettylib:MX_KAILH_SOCKET_WS2812_1U" H 4400 2500 60  0001 C CNN
+F 2 "prettylib:MX_KAILH_SOCKET_SK9822_1U" H 4400 2500 60  0001 C CNN
 F 3 "~" H 4400 2500 60  0000 C CNN
 	1    4400 2500
@@
 F 0 "S31" H 5100 2150 60  0000 C CNN
 F 1 "SW" H 5100 2000 60  0000 C CNN
-F 2 "prettylib:MX_KAILH_SOCKET_WS2812_1U" H 5100 2500 60  0001 C CNN
+F 2 "prettylib:MX_KAILH_SOCKET_SK9822_1U" H 5100 2500 60  0001 C CNN
 F 3 "~" H 5100 2500 60  0000 C CNN
 	1    5100 2500
@@
 F 0 "S35" H 5800 2150 60  0000 C CNN
 F 1 "SW" H 5800 2000 60  0000 C CNN
-F 2 "prettylib:MX_KAILH_SOCKET_WS2812_1U" H 5800 2500 60  0001 C CNN
+F 2 "prettylib:MX_KAILH_SOCKET_SK9822_1U" H 5800 2500 60  0001 C CNN
 F 3 "~" H 5800 2500 60  0000 C CNN
 	1    5800 2500
@@
 F 0 "S13" H 2300 2850 60  0000 C CNN
 F 1 "SW" H 2300 2700 60  0000 C CNN
-F 2 "prettylib:MX_KAILH_SOCKET_WS2812_1U" H 2300 3200 60  0001 C CNN
+F 2 "prettylib:MX_KAILH_SOCKET_SK9822_1U" H 2300 3200 60  0001 C CNN
 F 3 "~" H 2300 3200 60  0000 C CNN
 	1    2300 3200
@@
 F 0 "S18" H 3000 2850 60  0000 C CNN
 F 1 "SW" H 3000 2700 60  0000 C CNN
-F 2 "prettylib:MX_KAILH_SOCKET_WS2812_1U" H 3000 3200 60  0001 C CNN
+F 2 "prettylib:MX_KAILH_SOCKET_SK9822_1U" H 3000 3200 60  0001 C CNN
 F 3 "~" H 3000 3200 60  0000 C CNN
 	1    3000 3200
@@
 F 0 "S4" H 1600 1450 60  0000 C CNN
 F 1 "SW" H 1600 1300 60  0000 C CNN
-F 2 "prettylib:MX_KAILH_SOCKET_WS2812_1U" H 1600 1800 60  0001 C CNN
+F 2 "prettylib:MX_KAILH_SOCKET_SK9822_1U" H 1600 1800 60  0001 C CNN
 F 3 "~" H 1600 1800 60  0000 C CNN
 	1    1600 1800
@@
 F 0 "S33" H 5800 750 60  0000 C CNN
 F 1 "SW" H 5800 600 60  0000 C CNN
-F 2 "prettylib:MX_KAILH_SOCKET_WS2812_1U" H 5800 1100 60  0001 C CNN
+F 2 "prettylib:MX_KAILH_SOCKET_SK9822_1U" H 5800 1100 60  0001 C CNN
 F 3 "~" H 5800 1100 60  0000 C CNN
 	1    5800 1100

Commit message: Update YAEMK
Parts:
- D1, D10, D11, D12, D13, D14, D15, D16, D17, D18, D19, D2, D20, D21, D22, D23, D24, D25, D26, D27, D29, D3, D30, D31, D32, D34, D35, D36, D37, D4, D5, D6, D7, D9: footprint prettylib:D_SOD-323_HandSoldering -> Diode_SMD:D_SOD-123
- MH1, MH2, MH3, MH4, MH5, MH6, MH7, MH8, MH9: symbol YAEMK:Mounting_Hole -> YAEMK-rescue:Mounting_Hole-YAEMK
Changed lines of the file:
@@
 F 0 "D5" H 1800 1150 40  0000 C CNN
 F 1 "DIODE" H 1800 950 40  0000 C CNN
-F 2 "prettylib:D_SOD-323_HandSoldering" H 1800 1050 60  0001 C CNN
+F 2 "Diode_SMD:D_SOD-123" H 1800 1050 60  0001 C CNN
 F 3 "~" H 1800 1050 60  0000 C CNN
 	1    1800 1050
@@
 F 0 "D9" H 2500 1150 40  0000 C CNN
 F 1 "DIODE" H 2500 950 40  0000 C CNN
-F 2 "prettylib:D_SOD-323_HandSoldering" H 2500 1050 60  0001 C CNN
+F 2 "Diode_SMD:D_SOD-123" H 2500 1050 60  0001 C CNN
 F 3 "~" H 2500 1050 60  0000 C CNN
 	1    2500 1050
@@
 F 0 "D14" H 3200 1150 40  0000 C CNN
 F 1 "DIODE" H 3200 950 40  0000 C CNN
-F 2 "prettylib:D_SOD-323_HandSoldering" H 3200 1050 60  0001 C CNN
+F 2 "Diode_SMD:D_SOD-123" H 3200 1050 60  0001 C CNN
 F 3 "~" H 3200 1050 60  0000 C CNN
 	1    3200 1050
@@
 F 0 "D19" H 3900 1150 40  0000 C CNN
 F 1 "DIODE" H 3900 950 40  0000 C CNN
-F 2 "prettylib:D_SOD-323_HandSoldering" H 3900 1050 60  0001 C CNN
+F 2 "Diode_SMD:D_SOD-123" H 3900 1050 60  0001 C CNN
 F 3 "~" H 3900 1050 60  0000 C CNN
 	1    3900 1050
@@
 F 0 "D24" H 4600 1150 40  0000 C CNN
 F 1 "DIODE" H 4600 950 40  0000 C CNN
-F 2 "prettylib:D_SOD-323_HandSoldering" H 4600 1050 60  0001 C CNN
+F 2 "Diode_SMD:D_SOD-123" H 4600 1050 60  0001 C CNN
 F 3 "~" H 4600 1050 60  0000 C CNN
 	1    4600 1050
@@
 F 0 "D29" H 5300 1150 40  0000 C CNN
 F 1 "DIODE" H 5300 950 40  0000 C CNN
-F 2 "prettylib:D_SOD-323_HandSoldering" H 5300 1050 60  0001 C CNN
+F 2 "Diode_SMD:D_SOD-123" H 5300 1050 60  0001 C CNN
 F 3 "~" H 5300 1050 60  0000 C CNN
 	1    5300 1050
@@
 F 0 "D34" H 6000 1150 40  0000 C CNN
 F 1 "DIODE" H 6000 950 40  0000 C CNN
-F 2 "prettylib:D_SOD-323_HandSoldering" H 6000 1050 60  0001 C CNN
+F 2 "Diode_SMD:D_SOD-123" H 6000 1050 60  0001 C CNN
 F 3 "~" H 6000 1050 60  0000 C CNN
 	1    6000 1050
@@
 F 0 "D6" H 1800 1850 40  0000 C CNN
 F 1 "DIODE" H 1800 1650 40  0000 C CNN
-F 2 "prettylib:D_SOD-323_HandSoldering" H 1800 1750 60  0001 C CNN
+F 2 "Diode_SMD:D_SOD-123" H 1800 1750 60  0001 C CNN
 F 3 "~" H 1800 1750 60  0000 C CNN
 	1    1800 1750
@@
 F 0 "D10" H 2500 1850 40  0000 C CNN
 F 1 "DIODE" H 2500 1650 40  0000 C CNN
-F 2 "prettylib:D_SOD-323_HandSoldering" H 2500 1750 60  0001 C CNN
+F 2 "Diode_SMD:D_SOD-123" H 2500 1750 60  0001 C CNN
 F 3 "~" H 2500 1750 60  0000 C CNN
 	1    2500 1750
@@
 F 0 "D15" H 3200 1850 40  0000 C CNN
 F 1 "DIODE" H 3200 1650 40  0000 C CNN
-F 2 "prettylib:D_SOD-323_HandSoldering" H 3200 1750 60  0001 C CNN
+F 2 "Diode_SMD:D_SOD-123" H 3200 1750 60  0001 C CNN
 F 3 "~" H 3200 1750 60  0000 C CNN
 	1    3200 1750
@@
 F 0 "D20" H 3900 1850 40  0000 C CNN
 F 1 "DIODE" H 3900 1650 40  0000 C CNN
-F 2 "prettylib:D_SOD-323_HandSoldering" H 3900 1750 60  0001 C CNN
+F 2 "Diode_SMD:D_SOD-123" H 3900 1750 60  0001 C CNN
 F 3 "~" H 3900 1750 60  0000 C CNN
 	1    3900 1750
@@
 F 0 "D25" H 4600 1850 40  0000 C CNN
 F 1 "DIODE" H 4600 1650 40  0000 C CNN
-F 2 "prettylib:D_SOD-323_HandSoldering" H 4600 1750 60  0001 C CNN
+F 2 "Diode_SMD:D_SOD-123" H 4600 1750 60  0001 C CNN
 F 3 "~" H 4600 1750 60  0000 C CNN
 	1    4600 1750
@@
 F 0 "D30" H 5300 1850 40  0000 C CNN
 F 1 "DIODE" H 5300 1650 40  0000 C CNN
-F 2 "prettylib:D_SOD-323_HandSoldering" H 5300 1750 60  0001 C CNN
+F 2 "Diode_SMD:D_SOD-123" H 5300 1750 60  0001 C CNN
 F 3 "~" H 5300 1750 60  0000 C CNN
 	1    5300 1750
@@
 F 0 "D35" H 6000 1850 40  0000 C CNN
 F 1 "DIODE" H 6000 1650 40  0000 C CNN
-F 2 "prettylib:D_SOD-323_HandSoldering" H 6000 1750 60  0001 C CNN
+F 2 "Diode_SMD:D_SOD-123" H 6000 1750 60  0001 C CNN
 F 3 "~" H 6000 1750 60  0000 C CNN
 	1    6000 1750
@@
 F 0 "D11" H 2500 2550 40  0000 C CNN
 F 1 "DIODE" H 2500 2350 40  0000 C CNN
-F 2 "prettylib:D_SOD-323_HandSoldering" H 2500 2450 60  0001 C CNN
+F 2 "Diode_SMD:D_SOD-123" H 2500 2450 60  0001 C CNN
 F 3 "~" H 2500 2450 60  0000 C CNN
 	1    2500 2450
@@
 F 0 "D16" H 3200 2550 40  0000 C CNN
 F 1 "DIODE" H 3200 2350 40  0000 C CNN
-F 2 "prettylib:D_SOD-323_HandSoldering" H 3200 2450 60  0001 C CNN
+F 2 "Diode_SMD:D_SOD-123" H 3200 2450 60  0001 C CNN
 F 3 "~" H 3200 2450 60  0000 C CNN
 	1    3200 2450
@@
 F 0 "D21" H 3900 2550 40  0000 C CNN
 F 1 "DIODE" H 3900 2350 40  0000 C CNN
-F 2 "prettylib:D_SOD-323_HandSoldering" H 3900 2450 60  0001 C CNN
+F 2 "Diode_SMD:D_SOD-123" H 3900 2450 60  0001 C CNN
 F 3 "~" H 3900 2450 60  0000 C CNN
 	1    3900 2450
@@
 F 0 "D26" H 4600 2550 40  0000 C CNN
 F 1 "DIODE" H 4600 2350 40  0000 C CNN
-F 2 "prettylib:D_SOD-323_HandSoldering" H 4600 2450 60  0001 C CNN
+F 2 "Diode_SMD:D_SOD-123" H 4600 2450 60  0001 C CNN
 F 3 "~" H 4600 2450 60  0000 C CNN
 	1    4600 2450
@@
 F 0 "D31" H 5300 2550 40  0000 C CNN
 F 1 "DIODE" H 5300 2350 40  0000 C CNN
-F 2 "prettylib:D_SOD-323_HandSoldering" H 5300 2450 60  0001 C CNN
+F 2 "Diode_SMD:D_SOD-123" H 5300 2450 60  0001 C CNN
 F 3 "~" H 5300 2450 60  0000 C CNN
 	1    5300 2450
@@
 F 0 "D36" H 6000 2550 40  0000 C CNN
 F 1 "DIODE" H 6000 2350 40  0000 C CNN
-F 2 "prettylib:D_SOD-323_HandSoldering" H 6000 2450 60  0001 C CNN
+F 2 "Diode_SMD:D_SOD-123" H 6000 2450 60  0001 C CNN
 F 3 "~" H 6000 2450 60  0000 C CNN
 	1    6000 2450
@@
 F 0 "D1" H 1100 3250 40  0000 C CNN
 F 1 "DIODE" H 1100 3050 40  0000 C CNN
-F 2 "prettylib:D_SOD-323_HandSoldering" H 1100 3150 60  0001 C CNN
+F 2 "Diode_SMD:D_SOD-123" H 1100 3150 60  0001 C CNN
 F 3 "~" H 1100 3150 60  0000 C CNN
 	1    1100 3150
@@
 F 0 "D3" H 1800 3250 40  0000 C CNN
 F 1 "DIODE" H 1800 3050 40  0000 C CNN
-F 2 "prettylib:D_SOD-323_HandSoldering" H 1800 3150 60  0001 C CNN
+F 2 "Diode_SMD:D_SOD-123" H 1800 3150 60  0001 C CNN
 F 3 "~" H 1800 3150 60  0000 C CNN
 	1    1800 3150
@@
 F 0 "D12" H 2500 3250 40  0000 C CNN
 F 1 "DIODE" H 2500 3050 40  0000 C CNN
-F 2 "prettylib:D_SOD-323_HandSoldering" H 2500 3150 60  0001 C CNN
+F 2 "Diode_SMD:D_SOD-123" H 2500 3150 60  0001 C CNN
 F 3 "~" H 2500 3150 60  0000 C CNN
 	1    2500 3150
@@
 F 0 "D17" H 3200 3250 40  0000 C CNN
 F 1 "DIODE" H 3200 3050 40  0000 C CNN
-F 2 "prettylib:D_SOD-323_HandSoldering" H 3200 3150 60  0001 C CNN
+F 2 "Diode_SMD:D_SOD-123" H 3200 3150 60  0001 C CNN
 F 3 "~" H 3200 3150 60  0000 C CNN
 	1    3200 3150
@@
 F 0 "D22" H 3900 3250 40  0000 C CNN
 F 1 "DIODE" H 3900 3050 40  0000 C CNN
-F 2 "prettylib:D_SOD-323_HandSoldering" H 3900 3150 60  0001 C CNN
+F 2 "Diode_SMD:D_SOD-123" H 3900 3150 60  0001 C CNN
 F 3 "~" H 3900 3150 60  0000 C CNN
 	1    3900 3150
@@
 F 0 "D27" H 4600 3250 40  0000 C CNN
 F 1 "DIODE" H 4600 3050 40  0000 C CNN
-F 2 "prettylib:D_SOD-323_HandSoldering" H 4600 3150 60  0001 C CNN
+F 2 "Diode_SMD:D_SOD-123" H 4600 3150 60  0001 C CNN
 F 3 "~" H 4600 3150 60  0000 C CNN
 	1    4600 3150
@@
 F 0 "D32" H 5300 3250 40  0000 C CNN
 F 1 "DIODE" H 5300 3050 40  0000 C CNN
-F 2 "prettylib:D_SOD-323_HandSoldering" H 5300 3150 60  0001 C CNN
+F 2 "Diode_SMD:D_SOD-123" H 5300 3150 60  0001 C CNN
 F 3 "~" H 5300 3150 60  0000 C CNN
 	1    5300 3150
@@
 F 0 "D37" H 6000 3250 40  0000 C CNN
 F 1 "DIODE" H 6000 3050 40  0000 C CNN
-F 2 "prettylib:D_SOD-323_HandSoldering" H 6000 3150 60  0001 C CNN
+F 2 "Diode_SMD:D_SOD-123" H 6000 3150 60  0001 C CNN
 F 3 "~" H 6000 3150 60  0000 C CNN
 	1    6000 3150
@@
 F 0 "D2" H 1100 3950 40  0000 C CNN
 F 1 "DIODE" H 1100 3750 40  0000 C CNN
-F 2 "prettylib:D_SOD-323_HandSoldering" H 1100 3850 60  0001 C CNN
+F 2 "Diode_SMD:D_SOD-123" H 1100 3850 60  0001 C CNN
 F 3 "~" H 1100 3850 60  0000 C CNN
 	1    1100 3850
@@
 F 0 "D4" H 1800 3950 40  0000 C CNN
 F 1 "DIODE" H 1800 3750 40  0000 C CNN
-F 2 "prettylib:D_SOD-323_HandSoldering" H 1800 3850 60  0001 C CNN
+F 2 "Diode_SMD:D_SOD-123" H 1800 3850 60  0001 C CNN
 F 3 "~" H 1800 3850 60  0000 C CNN
 	1    1800 3850
@@
 F 0 "D13" H 2500 3950 40  0000 C CNN
 F 1 "DIODE" H 2500 3750 40  0000 C CNN
-F 2 "prettylib:D_SOD-323_HandSoldering" H 2500 3850 60  0001 C CNN
+F 2 "Diode_SMD:D_SOD-123" H 2500 3850 60  0001 C CNN
 F 3 "~" H 2500 3850 60  0000 C CNN
 	1    2500 3850
@@
 F 0 "D18" H 3200 3950 40  0000 C CNN
 F 1 "DIODE" H 3200 3750 40  0000 C CNN
-F 2 "prettylib:D_SOD-323_HandSoldering" H 3200 3850 60  0001 C CNN
+F 2 "Diode_SMD:D_SOD-123" H 3200 3850 60  0001 C CNN
 F 3 "~" H 3200 3850 60  0000 C CNN
 	1    3200 3850
@@
 F 0 "D7" H 1800 2550 40  0000 C CNN
 F 1 "DIODE" H 1800 2350 40  0000 C CNN
-F 2 "prettylib:D_SOD-323_HandSoldering" H 1800 2450 60  0001 C CNN
+F 2 "Diode_SMD:D_SOD-123" H 1800 2450 60  0001 C CNN
 F 3 "~" H 1800 2450 60  0000 C CNN
 	1    1800 2450
@@
 F 0 "D23" H 3900 3950 40  0000 C CNN
 F 1 "DIODE" H 3900 3750 40  0000 C CNN
-F 2 "prettylib:D_SOD-323_HandSoldering" H 3900 3850 60  0001 C CNN
+F 2 "Diode_SMD:D_SOD-123" H 3900 3850 60  0001 C CNN
 F 3 "~" H 3900 3850 60  0000 C CNN
 	1    3900 3850
@@
 Rot_Row
 $Comp
-L YAEMK:Mounting_Hole MH1
+L YAEMK-rescue:Mounting_Hole-YAEMK MH1
 U 1 1 5EF9B2DD
 P 7900 2400
@@
 $EndComp
 $Comp
-L YAEMK:Mounting_Hole MH2
+L YAEMK-rescue:Mounting_Hole-YAEMK MH2
 U 1 1 5EF9B5B8
 P 7900 800
@@
 $EndComp
 $Comp
-L YAEMK:Mounting_Hole MH3
+L YAEMK-rescue:Mounting_Hole-YAEMK MH3
 U 1 1 5EF9C683
 P 7900 2700
@@
 $EndComp
 $Comp
-L YAEMK:Mounting_Hole MH4
+L YAEMK-rescue:Mounting_Hole-YAEMK MH4
 U 1 1 5EF9D40E
 P 7900 1100
@@
 $EndComp
 $Comp
-L YAEMK:Mounting_Hole MH5
+L YAEMK-rescue:Mounting_Hole-YAEMK MH5
 U 1 1 5EF9E2EE
 P 7900 3000
@@
 $EndComp
 $Comp
-L YAEMK:Mounting_Hole MH6
+L YAEMK-rescue:Mounting_Hole-YAEMK MH6
 U 1 1 5EF9E2F8
 P 7900 1400
@@
 $EndComp
 $Comp
-L YAEMK:Mounting_Hole MH7
+L YAEMK-rescue:Mounting_Hole-YAEMK MH7
 U 1 1 5EF9E302
 P 7900 3300
@@
 $EndComp
 $Comp
-L YAEMK:Mounting_Hole MH8
+L YAEMK-rescue:Mounting_Hole-YAEMK MH8
 U 1 1 5EF9E30C
 P 7900 1700
@@
 $EndComp
 $Comp
-L YAEMK:Mounting_Hole MH9
+L YAEMK-rescue:Mounting_Hole-YAEMK MH9
 U 1 1 5F03D0F0
 P 7900 2050

Commit message: Sync
Connections:
- net labels added: VDD
- net labels removed: +5V
- wire segments 97 -> 96
Changed lines of the file:
@@
 Text GLabel 3600 6000 2    60   Input ~ 0
 Rot_B
-$Comp
-L YAEMK:+5V #PWR0101
-U 1 1 5EF4B6B0
-P 2300 5300
-F 0 "#PWR0101" H 2300 5390 20  0001 C CNN
-F 1 "+5V" H 2296 5428 30  0000 C CNN
-F 2 "" H 2300 5300 60  0000 C CNN
-F 3 "" H 2300 5300 60  0000 C CNN
-	1    2300 5300
-	1    0    0    -1
-$EndComp
 Wire Wire Line
 	2200 6900 2200 6800
@@
 	1800 6850 1800 6600
 Wire Wire Line
-	2300 5400 2200 5400
-Wire Wire Line
-	2300 5300 2300 5400
-Wire Wire Line
 	2200 6000 2200 5900
 Connection ~ 2200 6000
@@
 $EndComp
 Wire Wire Line
-	2400 5400 2300 5400
-Connection ~ 2300 5400
-Wire Wire Line
 	2400 5900 2400 6000
 Connection ~ 2400 6000
@@
 Text Notes 6950 600  0    50   ~ 0
 Mounting Hardware
+Wire Wire Line
+	2200 5400 2300 5400
+$Comp
+L YAEMK:VDD #PWR0101
+U 1 1 5FA3B535
+P 2300 5400
+F 0 "#PWR0101" H 2300 5500 30  0001 C CNN
+F 1 "VDD" H 2314 5538 30  0000 C CNN
+F 2 "" H 2300 5400 60  0000 C CNN
+F 3 "" H 2300 5400 60  0000 C CNN
+	1    2300 5400
+	1    0    0    -1
+$EndComp
+Connection ~ 2300 5400
+Wire Wire Line
+	2300 5400 2400 5400
 $EndSCHEMATC
