File: PCB/YAEMK.sch (KiCad schematic (older format))
At the start: 81 parts, among them SW1 ALPS EC11

Commit message: Merge Schematics
Parts:
- added C10, C11, C12, C13, C14, C15, C16, C17, C18, C19, C20, C21, C22, C23, C24, C25, C26, C27, C28, C29, C3, C30, C31, C32, C33, C34, C35, C37, C38, C39, C4, C40, C41, C42, C45, C48, C49, C5, C50, C51, C52, C53, C54, C6, C7, C8, C9: 100n, prettylib:SMD-0603, symbol YAEMK:C
- added C36, C43, C44: 10u, prettylib:SMD-0805, symbol YAEMK:C
- added C46, C47: 36p, prettylib:SMD-0603, symbol YAEMK:C
- added D35, D37, D38, D39, D40, D42, D44, D45, D46, D47, D48, D49, D50, D51, D52, D53, D54, D55, D56, D57, D58, D60, D61, D63, D64, D66, D67, D71, D72, D73, D74, D75, D76: SW, prettylib:SK6812_mini_e_flipable, symbol YAEMK:SK6812MINI-E
- added D36, D41, D43, D59, D62, D65: SW, prettylib:SK6812_mini_flipable, symbol YAEMK:SK6812MINI
- added D68, D69: 1N4148, prettylib:D_SOD-523, symbol YAEMK:DIODE
- added D70: LED, prettylib:LED-0603_flipable, symbol YAEMK:LED
- added D77: D_Schottky, prettylib:D_SOD-323_HandSoldering, symbol Device:D_Schottky
- added F1: 3A, prettylib:Fuse_1206_3216Metric, symbol Device:Polyfuse_Small
- added F2: 1.5A, prettylib:Fuse_1206_3216Metric, symbol Device:Polyfuse_Small
- added HSE1: 8MHz, prettylib:Crystal_SMD_3225-4Pin_3.2x2.5mm, symbol Device:Crystal_GND24_Small
- added J1: DBG, prettylib:PinHeader_1x06_P2.54mm_Horizontal, symbol YAEMK:CONN_6
- added JP1: LINK-, prettylib:SOLDER_JUMPER_3, symbol YAEMK:SolderJumper_3_Open
- added JP2: LINK+, prettylib:SOLDER_JUMPER_3, symbol YAEMK:SolderJumper_3_Open
- added L1: L_Core_Ferrite, prettylib:L_Taiyo-Yuden_MD-3030, symbol Device:L_Core_Ferrite
- added P1: PC, prettylib:USB_C_Receptacle_MUP_U22401, symbol YAEMK:USB_C_Receptacle_USB2.0
- added P2: Link, prettylib:USB_C_Receptacle_MUP_U22401, symbol YAEMK:USB_C_Receptacle_USB2.0
- added P3: SSD1107, prettylib:SSD1107_DISPLAY, symbol YAEMK:CONN_4
- added Q1: MMUN2133LT1G, prettylib:SOT-23, symbol Device:Q_PNP_BEC_BRT
- added R10, R9: 5.1k, prettylib:SMD-0603, symbol YAEMK:R
- added R11: 120, prettylib:SMD-0603, symbol YAEMK:R
- added R12, R13, R5, R6: 0, prettylib:SMD-0603, symbol YAEMK:R
- added R14: 1M, prettylib:SMD-0603, symbol YAEMK:R
- added R15: 450k, prettylib:SMD-0603, symbol YAEMK:R
- added R16, R23: 100k, prettylib:SMD-0603, symbol YAEMK:R
- added R17: 2k2, prettylib:SMD-0603, symbol YAEMK:R
- added R18, R19: 33, prettylib:SMD-0603, symbol YAEMK:R
- added R20, R7, R8: 1k5, prettylib:SMD-0603, symbol YAEMK:R
- added R21: 220, prettylib:SMD-0603, symbol YAEMK:R
- added R22, R26: 5k1, prettylib:SMD-0603, symbol YAEMK:R
- added R24, R25: 10k, prettylib:SMD-0603, symbol YAEMK:R
- added S32: DFU, prettylib:SMD_Tacticle_Switch_TS24CA_flipable, symbol YAEMK:SW
- added S33: NRST, prettylib:SMD_Tacticle_Switch_TS24CA_flipable, symbol YAEMK:SW
- added U1: 24LC64, prettylib:TSSOP-8_4.4x3mm_P0.65mm, symbol Memory_EEPROM:24LC64
- added U2: TLV62568DBVR, prettylib:SOT-23-5, symbol Regulator_Switching:TLV62568DBV
- added U3, U4: USBLC6-2SC6, prettylib:SOT-23-6_Handsoldering, symbol YAEMK:USBLC6-2SC6
- added U5: STM32F303CCTx, prettylib:LQFP-48_7x7mm_P0.5mm, symbol MCU_ST_STM32F3:STM32F303CCTx
Connections:
- net Col1: now also U5.12 (PA2)
- net Col2: now also U5.17 (PA7)
- net Col3: now also U5.18 (PB0)
- net Col4: now also U5.19 (PB1)
- net Col5: now also U5.20 (PB2)
- net Col6: now also U5.26 (PB13)
- net Col7: now also U5.27 (PB14)
- net Col8: now also U5.28 (PB15)
- net RGB_VDD: now also C10.1, C11.1, C12.1, C13.1, C14.1, C15.1, C16.1, C17.1, C18.1, C19.1, C20.1, C21.1, C22.1, C23.1, C24.1, C25.1, C26.1, C27.1, C28.1, C29.1, C3.1, C30.1, C31.1, C32.1, C33.1, C34.1, C35.1, C4.1, C43.1, C48.1, C49.1, C5.1, C50.1, C51.1, C52.1, C53.1, C6.1, C7.1, C8.1, C9.1, D35.1 (VDD), D36.4 (VDD), D37.1 (VDD), D38.1 (VDD), D39.1 (VDD), D40.1 (VDD), D41.4 (VDD), D42.1 (VDD), D43.4 (VDD), D44.1 (VDD), D45.1 (VDD), D46.1 (VDD), D47.1 (VDD), D48.1 (VDD), D49.1 (VDD), D50.1 (VDD), D51.1 (VDD), D52.1 (VDD), D53.1 (VDD), D54.1 (VDD), D55.1 (VDD), D56.1 (VDD), D57.1 (VDD), D58.1 (VDD), D59.4 (VDD), D60.1 (VDD), D61.1 (VDD), D62.4 (VDD), D63.1 (VDD), D64.1 (VDD), D65.4 (VDD), D66.1 (VDD), D67.1 (VDD), D71.1 (VDD), D72.1 (VDD), D73.1 (VDD), D74.1 (VDD), D75.1 (VDD), D76.1 (VDD), D77.1 (K), F2.2, R26.2, U2.1 (EN), U2.4 (VIN)
- net Rot_A: now also U5.13 (PA3)
- net Rot_B: now also U5.14 (PA4)
- net Row1: now also U5.29 (PA8)
- net Row2: now also U5.25 (PB12)
- net Row3: now also U5.16 (PA6)
- net Row4: now also U5.15 (PA5)
- net Row5: now also U5.11 (PA1)
- net VSS: now also C10.2, C11.2, C12.2, C13.2, C14.2, C15.2, C16.2, C17.2, C18.2, C19.2, C20.2, C21.2, C22.2, C23.2, C24.2, C25.2, C26.2, C27.2, C28.2, C29.2, C3.2, C30.2, C31.2, C32.2, C33.2, C34.2, C35.2, C36.2, C37.2, C38.2, C39.2, C4.2, C40.1, C41.2, C42.1, C43.2, C44.2, C45.1, C46.2, C47.2, C48.2, C49.2, C5.2, C50.2, C51.2, C52.2, C53.2, C54.2, C6.2, C7.2, C8.2, C9.2, D35.3 (VSS), D36.2 (VSS), D37.3 (VSS), D38.3 (VSS), D39.3 (VSS), D40.3 (VSS), D41.2 (VSS), D42.3 (VSS), D43.2 (VSS), D44.3 (VSS), D45.3 (VSS), D46.3 (VSS), D47.3 (VSS), D48.3 (VSS), D49.3 (VSS), D50.3 (VSS), D51.3 (VSS), D52.3 (VSS), D53.3 (VSS), D54.3 (VSS), D55.3 (VSS), D56.3 (VSS), D57.3 (VSS), D58.3 (VSS), D59.2 (VSS), D60.3 (VSS), D61.3 (VSS), D62.2 (VSS), D63.3 (VSS), D64.3 (VSS), D65.2 (VSS), D66.3 (VSS), D67.3 (VSS), D71.3 (VSS), D72.3 (VSS), D73.3 (VSS), D74.3 (VSS), D75.3 (VSS), D76.3 (VSS), HSE1.2, HSE1.4, J1.1, P1.A1 (GND), P1.A12 (GND), P1.B1 (GND), P1.B12 (GND), P2.A1 (GND), P2.A12 (GND), P2.B1 (GND), P2.B12 (GND), P3.4 (P4), R10.2, R12.1, R13.1, R14.2, R16.2, R17.2, R23.2, R25.2, R5.1, R6.1, R9.2, S32.2, S33.2, U1.1 (A0), U1.2 (A1), U1.3 (A2), U1.4 (GND), U1.7 (WP), U2.2 (GND), U3.2 (GND), U4.2 (GND), U5.23 (VSS), U5.35 (VSS), U5.47 (VSS), U5.8 (VSSA)
- new net: D45.2 (DOUT), D47.4 (DIN)
- new net: D43.1 (DOUT), D45.4 (DIN)
- new net: D51.2 (DOUT), D52.4 (DIN)
- new net: D50.2 (DOUT), D51.4 (DIN)
- new net: D56.2 (DOUT), D57.4 (DIN)
- new net: D55.2 (DOUT), D56.4 (DIN)
- new net: D61.2 (DOUT), D62.3 (DIN)
- new net: D60.2 (DOUT), D61.4 (DIN)
- new net: D47.2 (DOUT), D48.4 (DIN)
- new net: D52.2 (DOUT), D53.4 (DIN)
- new net: D57.2 (DOUT), D58.4 (DIN)
- new net: D38.2 (DOUT), D39.4 (DIN)
- new net: D37.2 (DOUT), D38.4 (DIN)
- new net: D43.3 (DIN), D44.2 (DOUT)
- new net: D48.2 (DOUT), D49.4 (DIN)
- new net: D53.2 (DOUT), D54.4 (DIN)
- new net: D63.2 (DOUT), D64.4 (DIN)
- new net: D62.1 (DOUT), D63.4 (DIN)
- new net: D44.4 (DIN), D46.2 (DOUT)
- new net: R18.2, U5.32 (PA11)
- new net: R19.2, U5.33 (PA12)
- new net: P1.B5 (CC2), R10.1
- new net: C47.1, HSE1.3, R21.2
- new net: P2.S1 (SHIELD), R12.2, R13.2
- new net: P1.S1 (SHIELD), R5.2, R6.2
- new net: D67.2 (DOUT), D71.4 (DIN)
- new net: D65.1 (DOUT), D67.4 (DIN)
- new net: D70.2 (K), R17.1
- new net: D68.2 (K), D69.2 (K), S32.1
- new net: R15.2, R16.1, U2.5 (FB)
- new net: D77.2 (A), F1.1, R22.1
- new net: Q1.3 (C), R11.1
- new net: P1.A5 (CC1), R9.1
- new net: L1.1, U2.3 (SW)
- new net: D35.2 (DOUT), D36.3 (DIN)
- new net: D40.2 (DOUT), D42.4 (DIN)
- new net: D39.2 (DOUT), D40.4 (DIN)
- new net: D49.2 (DOUT), D50.4 (DIN)
- new net: D54.2 (DOUT), D55.4 (DIN)
- new net: D59.1 (DOUT), D60.4 (DIN)
- new net: D65.3 (DIN), D66.2 (DOUT)
- new net: D64.2 (DOUT), D66.4 (DIN)
- new net: D36.1 (DOUT), D37.4 (DIN)
- new net: D41.1 (DOUT), D46.4 (DIN)
- new net: D41.3 (DIN), D42.2 (DOUT)
- new net: D58.2 (DOUT), D59.3 (DIN)
- new net: D75.2 (DOUT), D76.4 (DIN)
- new net: D74.2 (DOUT), D75.4 (DIN)
- new net: D73.2 (DOUT), D74.4 (DIN)
- new net: D72.2 (DOUT), D73.4 (DIN)
- new net: D71.2 (DOUT), D72.4 (DIN)
- new net BOOT0: C42.2, R11.2, R14.1, U5.44 (BOOT0)
- new net BOOT0_CHARGE: D68.1 (A), Q1.1 (B), U5.40 (PB4)
- new net ESD_LINK+: P2.A6 (D+), P2.B6 (D+), U4.3 (IO2)
- new net ESD_LINK-: P2.A7 (D-), P2.B7 (D-), U4.1 (IO1)
- new net ESD_USB_D+: P1.A6 (D+), P1.B6 (D+), U3.3 (IO2)
- new net ESD_USB_D-: P1.A7 (D-), P1.B7 (D-), U3.1 (IO1)
- new net HANDNESS: R24.2, R25.1, U5.2 (PC13)
- new net HSE_IN: C46.1, HSE1.1, U5.5 (PF0)
- new net HSE_OUT: R21.1, U5.6 (PF1)
- new net I2C1_SCL: P3.2 (P2), R8.2, U1.6 (SCL), U5.42 (PB6)
- new net I2C1_SDA: P3.1 (P1), R7.2, U1.5 (SDA), U5.43 (PB7)
- new net JTCK: J1.4, U5.37 (PA14)
- new net JTDI: J1.2, U5.38 (PA15)
- new net JTDO: J1.3, U5.39 (PB3)
- new net JTMS: J1.5, U5.34 (PA13)
- new net LINK+: JP2.2 (C), U4.4 (IO2)
- new net LINK-: JP1.2 (C), U4.6 (IO1)
- new net NRST: C40.2, D69.1 (A), S33.1, U5.7 (NRST)
- new net PLUG_DETECT: R22.2, R23.1, U5.30 (PA9)
- new net RGB_DATA: D35.4 (DIN), R26.1, U5.31 (PA10)
- new net USART3_RX: JP1.1 (A), JP2.1 (A), U5.22 (PB11)
- new net USART3_TX: JP1.3 (B), JP2.3 (B), U5.21 (PB10)
- new net USB_D+: R19.1, R20.1, U3.4 (IO2)
- new net USB_D-: R18.1, U3.6 (IO1)
- new net USB_VBUS: F1.2, P1.A4 (VBUS), P1.A9 (VBUS), P1.B4 (VBUS), P1.B9 (VBUS), U3.5 (VBUS)
- new net USB_VBUS_IN_FUSED: C45.2, F2.1, P2.A4 (VBUS), P2.A9 (VBUS), P2.B4 (VBUS), P2.B9 (VBUS), U4.5 (VBUS)
- new net VDD: C36.1, C37.1, C38.1, C39.1, C41.1, C44.1, C54.1, D70.1 (A), J1.6, L1.2, P3.3 (P3), Q1.2 (E), R15.1, R20.2, R24.1, R7.1, R8.1, U1.8 (VCC), U5.1 (VBAT), U5.24 (VDD), U5.36 (VDD), U5.48 (VDD), U5.9 (VDDA)
- no-connect marks 0 -> 13
Other:
- note added: "Board Link"
- note added: "CLOAD = 2 * (CLOAD_CRYSTAL - CPARASITIC)\n\nCPARASITIC = 2pF"
- note added: "Decoupling Capacitors"
- note added: "Display provides pull-up resistors"
- note added: "ESD protection"
- note added: "Fuses and plug detect"
- note added: "HSE Clock"
- note added: "Handness Selection"
- note added: "I2C EEPROM"
- note added: "Input Voltage Regulator"
- note added: "OLED Display"
- note added: "PC connection"
- note added: "Reset and DFU Bootloader Circuit"
- note added: "SWD / JTAG Interface\n"
- note added: "f(-3db) = 1 / (2 * pi * C * R)"
- moved on the sheet: C1, C2, D1, D10, D11, D12, D13, D14, D15, D16, D17, D18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

Commit message: Add Ideal Diode switch to LDO
Parts:
- removed D77: D_Schottky, prettylib:D_SOD-323_HandSoldering, symbol Device:D_Schottky
- removed L1: L_Core_Ferrite, prettylib:L_Taiyo-Yuden_MD-3030, symbol Device:L_Core_Ferrite
- removed R15: 450k, prettylib:SMD-0603, symbol YAEMK:R
- removed R16: 100k, prettylib:SMD-0603, symbol YAEMK:R
- removed U2: TLV62568DBVR, prettylib:SOT-23-5, symbol Regulator_Switching:TLV62568DBV
- added Q?: DMMT5401, Package_TO_SOT_SMD:SOT-23, symbol Transistor_FET:AO3401A
- added Q? (x2): DMMT5401, symbol Device:Q_DUAL_PNP_PNP_C1B1B2C2E2E1
- added R? (x2): 100k, prettylib:SMD-0603, symbol YAEMK:R
- added U?: SSP6206, prettylib:SOT-23, symbol YAEMK:SSP6206
- R22: value 5k1 -> 100k
Connections:
- wire segments 444 -> 453
Other:
- moved on the sheet: C43, C44, D70, F1, F2, R17, R22, R23
