File: PCB/YAEMK.sch (KiCad schematic (older format))
At the start: 217 parts, among them J1 DBG, P1 PC, P2 Link, P3 SSD1107, Q1 MMUN2133LT1G, Q2 DMMT5401, Q3 AO3401A, SW1 ALPS EC11, U1 24LC64, U2 SSP6206, U3 USBLC6-2SC6, U4 USBLC6-2SC6, U5 STM32F303CCTx

Commit message: Generate Gerbers and Add LCSC Part Numbers
Parts:
- C1, C10, C11, C12, C13, C14, C15, C16, C17, C18, C19, C2, C20, C21, C22, C23, C24, C25, C26, C27, C28, C29, C3, C30, C31, C32, C33, C34, C35, C36, C37, C38, C39, C4, C40, C41, C42, C45, C48, C49, C5, C50, C51, C52, C53, C54, C6, C7, C8, C9: JLCPCB BOM (none) -> 1; LCSC Part (none) -> C14663
- C43, C44: JLCPCB BOM (none) -> 1; LCSC Part (none) -> C15850
- C46, C47: value 36p -> 12p; JLCPCB BOM (none) -> 1; LCSC Part (none) -> C38523
- D1, D10, D11, D12, D13, D14, D15, D16, D17, D18, D19, D2, D20, D21, D22, D23, D24, D25, D26, D27, D28, D29, D3, D30, D31, D32, D33, D34, D4, D5, D6, D7, D8, D9: value DIODE -> 1N4148; JLCPCB BOM (none) -> 1; LCSC Part (none) -> C68948
- D35, D36, D37, D38, D39, D40, D41, D42, D43, D44, D45, D46, D47, D48, D49, D50, D51, D52, D53, D54, D55, D56, D57, D58, D59, D60, D61, D62, D63, D64, D65, D66, D67, D71, D72, D73, D74, D75, D76, D77, JP1, JP2, MH1, MH2, MH3, MH4, MH5, MH6, MH7, MH8, MH9, S1, S10, S11, S12, S13, S14, S15, S16, S17, S18, S19, S2, S20, S21, S22, S23, S24, S25, S26, S27, S28, S29, S3, S30, S31, S4, S5, S6, S7, S8, S9: JLCPCB BOM (none) -> 0
- D68, D69: JLCPCB BOM (none) -> 1; LCSC Part (none) -> C68948
- D70: JLCPCB BOM (none) -> 1; LCSC Part (none) -> C268294
- F1: JLCPCB BOM (none) -> 1; LCSC Part (none) -> C118413
- F2: JLCPCB BOM (none) -> 1; LCSC Part (none) -> C99563
- HSE1: JLCPCB BOM (none) -> 1; LCSC Part (none) -> C648984
- J1: JLCPCB BOM (none) -> 1; LCSC Part (none) -> C376124
- P1, P2: JLCPCB BOM (none) -> 1; LCSC Part (none) -> C168688
- P3: JLCPCB BOM (none) -> 1; LCSC Part (none) -> C358718
- Q1: JLCPCB BOM (none) -> 1; LCSC Part (none) -> C86182
- Q2: JLCPCB BOM (none) -> 1; LCSC Part (none) -> C154733
- Q3: JLCPCB BOM (none) -> 1; LCSC Part (none) -> C15127
- R1, R2, R24, R25, R3, R4: JLCPCB BOM (none) -> 1; LCSC Part (none) -> C25804
- R10, R9: value 5.1k -> 5k1; JLCPCB BOM (none) -> 1; LCSC Part (none) -> C23186
- R11: value 120 -> 220; JLCPCB BOM (none) -> 1; LCSC Part (none) -> C22962
- R12, R13, R5, R6: JLCPCB BOM (none) -> 1; LCSC Part (none) -> C21189
- R14: JLCPCB BOM (none) -> 1; LCSC Part (none) -> C22935
- R15, R16, R22, R23: JLCPCB BOM (none) -> 1; LCSC Part (none) -> C25803
- R17: JLCPCB BOM (none) -> 1; LCSC Part (none) -> C4190
- R18, R19: JLCPCB BOM (none) -> 1; LCSC Part (none) -> C23138
- R20, R7, R8: JLCPCB BOM (none) -> 1; LCSC Part (none) -> C22843
- R21: JLCPCB BOM (none) -> 1; LCSC Part (none) -> C22962
- R26: JLCPCB BOM (none) -> 1; LCSC Part (none) -> C23186
- S32, S33: JLCPCB BOM (none) -> 1; LCSC Part (none) -> C393942
- SW1: JLCPCB BOM (none) -> 1; LCSC Part (none) -> C370986
- U1: JLCPCB BOM (none) -> 1; LCSC Part (none) -> C189763
- U2: JLCPCB BOM (none) -> 1; LCSC Part (none) -> C5446
- U3, U4: JLCPCB BOM (none) -> 1; LCSC Part (none) -> C7519
- U5: JLCPCB BOM (none) -> 1; LCSC Part (none) -> C81523

Commit message: Add assembly holes for real
Parts:
- added MH10, MH11, MH12: MOUNT_HOLE, prettylib:JLC_SMT_Assembly_Hole, symbol YAEMK:MOUNT_HOLE
Changed lines of the file:
@@
 	0    1    1    0
 $EndComp
+$Comp
+L YAEMK:MOUNT_HOLE MH10
+U 1 1 5FFBE911
+P 20550 7600
+F 0 "MH10" H 20678 7653 60  0000 L CNN
+F 1 "MOUNT_HOLE" H 20678 7547 60  0000 L CNN
+F 2 "prettylib:JLC_SMT_Assembly_Hole" H 20550 7600 60  0001 C CNN
+F 3 "" H 20550 7600 60  0000 C CNN
+	1    20550 7600
+	1    0    0    -1
+$EndComp
+$Comp
+L YAEMK:MOUNT_HOLE MH11
+U 1 1 5FFC070F
+P 20550 7900
+F 0 "MH11" H 20678 7953 60  0000 L CNN
+F 1 "MOUNT_HOLE" H 20678 7847 60  0000 L CNN
+F 2 "prettylib:JLC_SMT_Assembly_Hole" H 20550 7900 60  0001 C CNN
+F 3 "" H 20550 7900 60  0000 C CNN
+	1    20550 7900
+	1    0    0    -1
+$EndComp
+$Comp
+L YAEMK:MOUNT_HOLE MH12
+U 1 1 5FFC25D4
+P 20550 8250
+F 0 "MH12" H 20678 8303 60  0000 L CNN
+F 1 "MOUNT_HOLE" H 20678 8197 60  0000 L CNN
+F 2 "prettylib:JLC_SMT_Assembly_Hole" H 20550 8250 60  0001 C CNN
+F 3 "" H 20550 8250 60  0000 C CNN
+	1    20550 8250
+	1    0    0    -1
+$EndComp
 $EndSCHEMATC

Commit message: Add logos as symbols, clean up symbols
Parts:
- added G1, G2: Logo, prettylib:LOGO, symbol YAEMK:Logo
- MH10, MH11, MH12: value MOUNT_HOLE -> Assembly Hole; symbol YAEMK:MOUNT_HOLE -> YAEMK:Assembly_Hole
Changed lines of the file:
@@
 Wire Wire Line
 	3700 14100 3700 14300
-Text GLabel 5050 11600 2    50   Input ~ 0
+Text GLabel 1750 9850 2    50   Input ~ 0
 RGB_VDD
-Text GLabel 4900 11600 0    50   Input ~ 0
+Text GLabel 1600 9850 0    50   Input ~ 0
 USB_VBUS_IN
 Wire Wire Line
-	4900 11600 5050 11600
+	1600 9850 1750 9850
 Wire Wire Line
 	10300 13250 10900 13250
@@
 $EndComp
 $Comp
-L YAEMK:MOUNT_HOLE MH10
+L YAEMK:Assembly_Hole MH10
 U 1 1 5FFBE911
-P 20550 7600
-F 0 "MH10" H 20678 7653 60  0000 L CNN
-F 1 "MOUNT_HOLE" H 20678 7547 60  0000 L CNN
-F 2 "prettylib:JLC_SMT_Assembly_Hole" H 20550 7600 60  0001 C CNN
-F 3 "" H 20550 7600 60  0000 C CNN
-	1    20550 7600
-	1    0    0    -1
-$EndComp
-$Comp
-L YAEMK:MOUNT_HOLE MH11
+P 19950 7550
+F 0 "MH10" H 20078 7603 60  0000 L CNN
+F 1 "Assembly Hole" H 20078 7497 60  0000 L CNN
+F 2 "prettylib:JLC_SMT_Assembly_Hole" H 19950 7550 60  0001 C CNN
+F 3 "" H 19950 7550 60  0000 C CNN
+	1    19950 7550
+	1    0    0    -1
+$EndComp
+$Comp
+L YAEMK:Assembly_Hole MH11
 U 1 1 5FFC070F
-P 20550 7900
-F 0 "MH11" H 20678 7953 60  0000 L CNN
-F 1 "MOUNT_HOLE" H 20678 7847 60  0000 L CNN
-F 2 "prettylib:JLC_SMT_Assembly_Hole" H 20550 7900 60  0001 C CNN
-F 3 "" H 20550 7900 60  0000 C CNN
-	1    20550 7900
-	1    0    0    -1
-$EndComp
-$Comp
-L YAEMK:MOUNT_HOLE MH12
+P 19950 7850
+F 0 "MH11" H 20078 7903 60  0000 L CNN
+F 1 "Assembly Hole" H 20078 7797 60  0000 L CNN
+F 2 "prettylib:JLC_SMT_Assembly_Hole" H 19950 7850 60  0001 C CNN
+F 3 "" H 19950 7850 60  0000 C CNN
+	1    19950 7850
+	1    0    0    -1
+$EndComp
+$Comp
+L YAEMK:Assembly_Hole MH12
 U 1 1 5FFC25D4
-P 20550 8250
-F 0 "MH12" H 20678 8303 60  0000 L CNN
-F 1 "MOUNT_HOLE" H 20678 8197 60  0000 L CNN
-F 2 "prettylib:JLC_SMT_Assembly_Hole" H 20550 8250 60  0001 C CNN
-F 3 "" H 20550 8250 60  0000 C CNN
-	1    20550 8250
-	1    0    0    -1
-$EndComp
+P 19950 8200
+F 0 "MH12" H 20078 8253 60  0000 L CNN
+F 1 "Assembly Hole" H 20078 8147 60  0000 L CNN
+F 2 "prettylib:JLC_SMT_Assembly_Hole" H 19950 8200 60  0001 C CNN
+F 3 "" H 19950 8200 60  0000 C CNN
+	1    19950 8200
+	1    0    0    -1
+$EndComp
+$Comp
+L YAEMK:Logo G1
+U 1 1 5FE39567
+P 20150 8900
+F 0 "G1" H 20150 9134 50  0000 C CNN
+F 1 "Logo" H 20150 9043 50  0000 C CNN
+F 2 "prettylib:LOGO" H 20150 8900 50  0001 C CNN
+F 3 "" H 20150 8900 50  0001 C CNN
+	1    20150 8900
+	1    0    0    -1
+$EndComp
+$Comp
+L YAEMK:Logo G2
+U 1 1 5FE3B26E
+P 20150 9350
+F 0 "G2" H 20150 9584 50  0000 C CNN
+F 1 "Logo" H 20150 9493 50  0000 C CNN
+F 2 "prettylib:LOGO" H 20150 9350 50  0001 C CNN
+F 3 "" H 20150 9350 50  0001 C CNN
+	1    20150 9350
+	1    0    0    -1
+$EndComp

Commit message: Remove WS2812 from mx symbols
Parts:
- S1, S5: symbol YAEMK:MX_WS2812_2U_2X1U -> YAEMK:MX_2U_2X1U
- S10, S11, S12, S13, S14, S15, S16, S17, S18, S19, S2, S20, S21, S22, S23, S24, S25, S26, S27, S28, S29, S3, S30, S31, S4, S6, S7, S8, S9: symbol YAEMK:MX_WS2812_1U -> YAEMK:MX_1U
Changed lines of the file:
@@
 $EndDescr
 $Comp
-L YAEMK:MX_WS2812_1U S2
+L YAEMK:MX_1U S2
 U 1 1 549A1D53
 P 1900 600
@@
 $EndComp
 $Comp
-L YAEMK:MX_WS2812_1U S6
+L YAEMK:MX_1U S6
 U 1 1 549A1D79
 P 2600 600
@@
 $EndComp
 $Comp
-L YAEMK:MX_WS2812_1U S11
+L YAEMK:MX_1U S11
 U 1 1 549A1D85
 P 3300 600
@@
 $EndComp
 $Comp
-L YAEMK:MX_WS2812_1U S16
+L YAEMK:MX_1U S16
 U 1 1 549A1D91
 P 4000 600
@@
 $EndComp
 $Comp
-L YAEMK:MX_WS2812_1U S20
+L YAEMK:MX_1U S20
 U 1 1 549A1D9D
 P 4700 600
@@
 $EndComp
 $Comp
-L YAEMK:MX_WS2812_1U S24
+L YAEMK:MX_1U S24
 U 1 1 549A1DA9
 P 5400 600
@@
 $EndComp
 $Comp
-L YAEMK:MX_WS2812_1U S28
+L YAEMK:MX_1U S28
 U 1 1 549A1DB5
 P 6100 600
@@
 $EndComp
 $Comp
-L YAEMK:MX_WS2812_1U S3
+L YAEMK:MX_1U S3
 U 1 1 549A1DC1
 P 1900 1300
@@
 $EndComp
 $Comp
-L YAEMK:MX_WS2812_1U S7
+L YAEMK:MX_1U S7
 U 1 1 549A1DCD
 P 2600 1300
@@
 $EndComp
 $Comp
-L YAEMK:MX_WS2812_1U S12
+L YAEMK:MX_1U S12
 U 1 1 549A1DD9
 P 3300 1300
@@
 $EndComp
 $Comp
-L YAEMK:MX_WS2812_1U S17
+L YAEMK:MX_1U S17
 U 1 1 549A1DE5
 P 4000 1300
@@
 $EndComp
 $Comp
-L YAEMK:MX_WS2812_1U S21
+L YAEMK:MX_1U S21
 U 1 1 549A1DF1
 P 4700 1300
@@
 $EndComp
 $Comp
-L YAEMK:MX_WS2812_1U S25
+L YAEMK:MX_1U S25
 U 1 1 549A1DFD
 P 5400 1300
@@
 $EndComp
 $Comp
-L YAEMK:MX_WS2812_1U S8
+L YAEMK:MX_1U S8
 U 1 1 549A1E15
 P 2600 2000
@@
 $EndComp
 $Comp
-L YAEMK:MX_WS2812_1U S13
+L YAEMK:MX_1U S13
 U 1 1 549A1E21
 P 3300 2000
@@
 $EndComp
 $Comp
-L YAEMK:MX_WS2812_1U S18
+L YAEMK:MX_1U S18
 U 1 1 549A1E2D
 P 4000 2000
@@
 $EndComp
 $Comp
-L YAEMK:MX_WS2812_1U S22
+L YAEMK:MX_1U S22
 U 1 1 549A1E39
 P 4700 2000
@@
 $EndComp
 $Comp
-L YAEMK:MX_WS2812_1U S26
+L YAEMK:MX_1U S26
 U 1 1 549A1E45
 P 5400 2000
@@
 $EndComp
 $Comp
-L YAEMK:MX_WS2812_1U S30
+L YAEMK:MX_1U S30
 U 1 1 549A1E51
 P 6100 2000
@@
 $EndComp
 $Comp
-L YAEMK:MX_WS2812_1U S9
+L YAEMK:MX_1U S9
 U 1 1 549A1E81
 P 2600 2700
@@
 $EndComp
 $Comp
-L YAEMK:MX_WS2812_1U S14
+L YAEMK:MX_1U S14
 U 1 1 549A1E8D
 P 3300 2700
@@
 $EndComp
 $Comp
-L YAEMK:MX_WS2812_1U S19
+L YAEMK:MX_1U S19
 U 1 1 549A1E99
 P 4000 2700
@@
 $EndComp
 $Comp
-L YAEMK:MX_WS2812_1U S23
+L YAEMK:MX_1U S23
 U 1 1 549A1EA5
 P 4700 2700
@@
 $EndComp
 $Comp
-L YAEMK:MX_WS2812_1U S27
+L YAEMK:MX_1U S27
 U 1 1 549A1EB1
 P 5400 2700
@@
 $EndComp
 $Comp
-L YAEMK:MX_WS2812_1U S31
+L YAEMK:MX_1U S31
 U 1 1 549A1EBD
 P 6100 2700
@@
 $EndComp
 $Comp
-L YAEMK:MX_WS2812_1U S10
+L YAEMK:MX_1U S10
 U 1 1 549A1EED
 P 2600 3400
@@
 $EndComp
 $Comp
-L YAEMK:MX_WS2812_1U S15
+L YAEMK:MX_1U S15
 U 1 1 549A1EF9
 P 3300 3400
@@
 Switch Matrix
 $Comp
-L YAEMK:MX_WS2812_2U_2X1U S1
+L YAEMK:MX_2U_2X1U S1
 U 1 1 5F0DAADF
 P 1200 2850
@@
 $EndComp
 $Comp
-L YAEMK:MX_WS2812_2U_2X1U S1
+L YAEMK:MX_2U_2X1U S1
 U 2 1 5F0DFACD
 P 1200 3500
@@
 	1700 1750 1700 2450
 $Comp
-L YAEMK:MX_WS2812_1U S4
+L YAEMK:MX_1U S4
 U 1 1 549A1E75
 P 1900 2000
@@
 	850  5150 7150 5150
 $Comp
-L YAEMK:MX_WS2812_1U S29
+L YAEMK:MX_1U S29
 U 1 1 549A1E09
 P 6100 1300
@@
 $EndComp
 $Comp
-L YAEMK:MX_WS2812_2U_2X1U S5
+L YAEMK:MX_2U_2X1U S5
 U 2 1 5F0E7608
 P 1900 3500
@@
 $EndComp
 $Comp
-L YAEMK:MX_WS2812_2U_2X1U S5
+L YAEMK:MX_2U_2X1U S5
 U 1 1 5F0E0C97
 P 1900 2850
